File: anderson_pp_input.kicad_sch (KiCad schematic)
At the start: 10 parts, among them J3 1377G12-BK, J4 MCV 1,5/ 2-GF-3,81, Q5 AO3400A, U4 LM74610

Commit message: library rename
Parts:
- F3: footprint gx_lib:MCCQ-122 -> kicad_gx_library:Fuse_MCCQ-122
- J3: footprint gx_lib:Anderson_PP25_RA_1377g12-bk -> kicad_gx_library:Connector_Anderson_PP25_RA_1377g12-bk
- U4: symbol _gxLib:LM74610 -> kicad_gx_library:LM74610
Changed lines of the file:
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@@
 			)
 		)
-		(property "Footprint" "gx_lib:MCCQ-122"
+		(property "Footprint" "kicad_gx_library:Fuse_MCCQ-122"
 			(at 73.66 81.788 90)
 			(hide yes)
@@
 			)
 		)
-		(property "Footprint" "gx_lib:Anderson_PP25_RA_1377g12-bk"
+		(property "Footprint" "kicad_gx_library:Connector_Anderson_PP25_RA_1377g12-bk"
 			(at 39.37 63.5 0)
 			(hide yes)
@@
 	)
 	(symbol
-		(lib_id "_gxLib:LM74610")
+		(lib_id "kicad_gx_library:LM74610")
 		(at 148.59 78.74 0)
 		(unit 1)
@@
 		(fields_autoplaced yes)
 		(property "Reference" "U4"
-			(at 162.56 100.2598 0)
+			(at 165.1 97.7198 0)
 			(show_name no)
 			(do_not_autoplace no)
@@
 		)
 		(property "Value" "LM74610"
-			(at 148.59 78.74 0)
-			(show_name no)
-			(do_not_autoplace no)
+			(at 165.1 100.2598 0)
+			(show_name no)
+			(do_not_autoplace no)
