File: anderson_pp_input.kicad_sch (KiCad schematic)
At the start: 10 parts, among them J3 1377G12-BK, J4 MCV 1,5/ 2-GF-3,81, Q5 AO3400A, U4 LM74610

Commit message: hierarchy
Parts:
- removed C9: 1u/16V, Capacitor_SMD:C_0805_2012Metric, symbol Device:C_Small
- removed D2: SMAJ18A, Diode_SMD:D_SMA, symbol Diode:SMAJ18A
- removed F3: Fuse 2A, kicad_gx_library:Fuse_MCCQ-122, symbol Device:Fuse
- removed J3: 1377G12-BK, kicad_gx_library:Connector_Anderson_PP25_RA_1377g12-bk, symbol Connector_Generic:Conn_01x02
- removed J4: MCV 1,5/ 2-GF-3,81, Connector_Phoenix_MC:PhoenixContact_MCV_1,5_2-GF-3.81_1x02_P3.81mm_Vertical_ThreadedFlange_MountHole, symbol Connector_Generic:Conn_01x02
- removed JP7, JP8: SolderJumper_2_Open, Jumper:SolderJumper-2_P1.3mm_Open_TrianglePad1.0x1.5mm, symbol Jumper:SolderJumper_2_Open
- removed Q5: AO3400A, Package_TO_SOT_SMD:SOT-23, symbol Transistor_FET:AO3400A
- removed TP4: TestPoint, TestPoint:TestPoint_Pad_D1.5mm, symbol Connector:TestPoint
- removed U4: LM74610, Package_SO:VSSOP-8_3x3mm_P0.65mm, symbol kicad_gx_library:LM74610
Other:
- note removed: "X7R 0805"
