File: foxhunt1.kicad_pcb (KiCad board)
At the start: 2 copper layers, 51 parts, among them J3 1377G12-BK, J4 MCV 1,5/ 2-GF-3,81, Q1 AO3400A, Q2 8205A, Q3 AO3400A, Q5 AO3400A, U2 TPS563201, U3 LM74610, U4 LM74610, U5 LM1085-5.0

Commit message: library rename
Parts:
- removed C15: 22u/16V, Capacitor_SMD:C_1206_3216Metric
- added C16: 0.1u/25V, Capacitor_SMD:C_0603_1608Metric, F.Cu at (68.4, 152.5)
- added C17: 10u/25V, Capacitor_SMD:C_0805_2012Metric, F.Cu at (48.1, 161.6)
- added C18: 10u/25V, Capacitor_SMD:C_0805_2012Metric, F.Cu at (48.1, 164.6)
- added C19: 0.1u/25V, Capacitor_SMD:C_0603_1608Metric, F.Cu at (68.4, 155.0)
- added C20: 22u/16V, Capacitor_SMD:C_1206_3216Metric, F.Cu at (48.7, 155.1)
- added C21: 22u/16V, Capacitor_SMD:C_1206_3216Metric, F.Cu at (48.7, 158.4)
- added C22: 0.1u/25V, Capacitor_SMD:C_0603_1608Metric, F.Cu at (68.4, 157.5)
- added C23: 22u/16V Elec, Capacitor_SMD:C_Elec_5x5.8, F.Cu at (56.8, 140.9)
- added C24: 22u/16V Elec, Capacitor_SMD:C_Elec_5x5.8, F.Cu at (56.8, 147.8)
- added C25: 0.1u/25V, Capacitor_SMD:C_0603_1608Metric, F.Cu at (68.4, 160.0)
- added JP1: Jumper_2_Open, TestPoint:TestPoint_2Pads_Pitch2.54mm_Drill0.8mm, F.Cu at (54.4, 160.7)
- added JP11: SolderJumper_2_Open, Jumper:SolderJumper-2_P1.3mm_Open_TrianglePad1.0x1.5mm, F.Cu at (64.3, 160.1)
- added JP12: SolderJumper_2_Open, Jumper:SolderJumper-2_P1.3mm_Open_TrianglePad1.0x1.5mm, F.Cu at (64.3, 163.6)
- added JP4: SolderJumper_2_Open, Jumper:SolderJumper-2_P1.3mm_Open_TrianglePad1.0x1.5mm, F.Cu at (64.3, 153.0)
- added JP5: SolderJumper_2_Open, Jumper:SolderJumper-2_P1.3mm_Open_TrianglePad1.0x1.5mm, F.Cu at (64.3, 156.5)
- added JP6: Jumper_2_Open, TestPoint:TestPoint_2Pads_Pitch2.54mm_Drill0.8mm, F.Cu at (54.4, 164.1)
- added L2: 3.3uH, kicad_gx_library:L_Chilisin_MHCI06030, F.Cu at (57.3, 155.1)
- added R11: 10k, Resistor_SMD:R_0805_2012Metric, F.Cu at (43.7, 154.9)
- added R12: 10k, Resistor_SMD:R_0805_2012Metric, F.Cu at (43.7, 157.8)
- added R13: 46.4k, Resistor_SMD:R_0805_2012Metric, F.Cu at (43.7, 160.8)
- added R14: 16.5 2W, Resistor_THT:R_Axial_Power_L20.0mm_W6.4mm_P5.08mm_Vertical, F.Cu at (45.5, 141.5)
- added R15: 24.9 2W, Resistor_THT:R_Axial_Power_L20.0mm_W6.4mm_P5.08mm_Vertical, F.Cu at (45.5, 149.4)
- added U6: TPS563201, Package_TO_SOT_SMD:SOT-23-6, F.Cu at (63.6, 148.2)
- added U7: AMS1117-3.3, Package_TO_SOT_SMD:SOT-223-3_TabPin2, F.Cu at (65.9, 141.7)
- F2: footprint gx_lib:PTCC_CLM1612 -> kicad_gx_library:Fuse_PTCC_CLM1612
- F3: footprint gx_lib:MCCQ-122 -> kicad_gx_library:Fuse_MCCQ-122
- J3: footprint gx_lib:Anderson_PP25_RA_1377g12-bk -> kicad_gx_library:Connector_Anderson_PP25_RA_1377g12-bk
- L1: footprint gx_lib:L_Chilisin_MHCI06030 -> kicad_gx_library:L_Chilisin_MHCI06030
Connections:
- BT2 pad 2: GND -> GNDREF
- C2 pad 2: GND -> GNDREF
- C3 pad 2: GND -> GNDREF
- C4 pad 2: GND -> GNDREF
- C5 pad 2: GND -> GNDREF
- C6 pad 2: GND -> GNDREF
- Q1 pad 2: GND -> GNDREF
- R3 pad 1: GND -> GNDREF
- TH1 pad 2: GND -> GNDREF
- U1 pad 20: GND -> GNDREF
- U1 pad 25: GND -> GNDREF
- U5 pad 2: +5V -> Net-(JP11-A)
