File: foxhunt1.kicad_pcb (KiCad board)
At the start: 2 copper layers, 74 parts, among them J3 1377G12-BK, J4 MCV 1,5/ 2-GF-3,81, Q1 AO3400A, Q2 8205A, Q3 AO3400A, Q5 AO3400A, U2 TPS563201, U3 LM74610, U4 LM74610, U5 LM1085-5.0, U6 TPS563201, U7 AMS1117-3.3

Commit message: Make project library-portable; fix Q2 footprint reference
Vendor the three non-standard libraries (kicad_gx_library,
digikey-kicad-library, SparkFun-KiCad-Libraries) as git submodules
under libs/, and add project-level sym-lib-table/fp-lib-table entries
that resolve them via ${KIPRJMOD}, so the project no longer depends on
this machine's global KiCad library setup.

Also fixes Q2's footprint reference, which pointed at an unregistered
"DigikeyGithub" library nickname left over from a prior library setup;
it now correctly resolves to digikey-kicad-library:SOT23-6L.

Co-Authored-By: Claude Sonnet 5 <noreply@anthropic.com>
Parts:
- Q2: footprint DigikeyGithub:SOT23-6L -> digikey-kicad-library:SOT23-6L
Changed lines of the file:
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@@
 		(embedded_fonts no)
 	)
-	(footprint "DigikeyGithub:SOT23-6L"
+	(footprint "digikey-kicad-library:SOT23-6L"
 		(layer "F.Cu")
 		(at 145.54 112.575)
