File: foxhunt1.kicad_pcb (KiCad board)
At the start: 2 copper layers, 74 parts, among them J3 1377G12-BK, J4 MCV 1,5/ 2-GF-3,81, Q1 AO3400A, Q2 8205A, Q3 AO3400A, Q5 AO3400A, U2 TPS563201, U3 LM74610, U4 LM74610, U5 LM1085-5.0, U6 TPS563201, U7 AMS1117-3.3

Commit message: hierarchy work
Parts:
- removed C10, C22, C25: 0.1u/25V, Capacitor_SMD:C_0603_1608Metric
- removed C17: 10u/25V, Capacitor_SMD:C_0805_2012Metric
- removed C20, C21: 22u/16V, Capacitor_SMD:C_1206_3216Metric
- removed C23, C24: 22u/16V Elec, Capacitor_SMD:C_Elec_5x5.8
- removed C9: 1u/16V, Capacitor_SMD:C_0805_2012Metric
- removed JP1, JP6: Jumper_2_Open, TestPoint:TestPoint_2Pads_Pitch2.54mm_Drill0.8mm
- removed JP11, JP2, JP3, JP4, JP5, JP7: SolderJumper_2_Open, Jumper:SolderJumper-2_P1.3mm_Open_TrianglePad1.0x1.5mm
- removed L1, L2: 3.3uH, kicad_gx_library:L_Chilisin_MHCI06030
- removed Q3, Q5: AO3400A, Package_TO_SOT_SMD:SOT-23
- removed R14: 16.5 2W, Resistor_THT:R_Axial_Power_L20.0mm_W6.4mm_P5.08mm_Vertical
- removed R15: 24.9 2W, Resistor_THT:R_Axial_Power_L20.0mm_W6.4mm_P5.08mm_Vertical
- removed U4: LM74610, Package_SO:VSSOP-8_3x3mm_P0.65mm
- removed U5: LM1085-5.0, Package_TO_SOT_SMD:TO-263-3_TabPin2
- removed U6: TPS563201, Package_TO_SOT_SMD:SOT-23-6
- added C15: 0.1u/25V, Capacitor_SMD:C_0603_1608Metric, F.Cu at (47.0, 130.5)
- added C28: 22u/16V, Capacitor_SMD:C_1206_3216Metric, F.Cu at (52.2, 118.0)
- added C29: 22u/16V, Capacitor_SMD:C_1206_3216Metric, F.Cu at (52.2, 121.4)
- added C30: 22u/16V, Capacitor_SMD:C_1206_3216Metric, F.Cu at (52.2, 124.7)
- added C31: 22u/16V, Capacitor_SMD:C_1206_3216Metric, F.Cu at (52.2, 128.1)
- added C32: 0.1u/25V, Capacitor_SMD:C_0603_1608Metric, F.Cu at (47.0, 133.0)
- added C33: 0.1u/25V, Capacitor_SMD:C_0603_1608Metric, F.Cu at (47.0, 135.6)
- added C34: 0.1u/25V, Capacitor_SMD:C_0603_1608Metric, F.Cu at (47.0, 138.1)
- added C35: 0.1u/25V, Capacitor_SMD:C_0603_1608Metric, F.Cu at (47.0, 140.6)
- added C36: 22u/16V Elec, Capacitor_SMD:C_Elec_5x5.8, F.Cu at (78.6, 103.9)
- added C37: 22u/16V Elec, Capacitor_SMD:C_Elec_5x5.8, F.Cu at (78.6, 110.7)
- added JP13: SolderJumper_2_Open, Jumper:SolderJumper-2_P1.3mm_Open_TrianglePad1.0x1.5mm, F.Cu at (47.2, 109.3)
- added JP14: SolderJumper_2_Open, Jumper:SolderJumper-2_P1.3mm_Open_TrianglePad1.0x1.5mm, F.Cu at (47.2, 112.9)
- added JP15: Jumper_2_Open, TestPoint:TestPoint_2Pads_Pitch2.54mm_Drill0.8mm, F.Cu at (66.7, 130.4)
- added JP16: Jumper_2_Open, TestPoint:TestPoint_2Pads_Pitch2.54mm_Drill0.8mm, F.Cu at (66.7, 133.7)
- added JP17: SolderJumper_2_Open, Jumper:SolderJumper-2_P1.3mm_Open_TrianglePad1.0x1.5mm, F.Cu at (47.2, 116.4)
- added JP18: SolderJumper_2_Open, Jumper:SolderJumper-2_P1.3mm_Open_TrianglePad1.0x1.5mm, F.Cu at (47.2, 120.0)
- added JP20: SolderJumper_2_Open, Jumper:SolderJumper-2_P1.3mm_Open_TrianglePad1.0x1.5mm, F.Cu at (133.5, 111.1)
- added JP21: SolderJumper_2_Open, Jumper:SolderJumper-2_P1.3mm_Open_TrianglePad1.0x1.5mm, F.Cu at (133.5, 114.7)
- added L3: 3.3uH, kicad_gx_library:L_Chilisin_MHCI06030, F.Cu at (65.2, 104.4)
- added L4: 3.3uH, kicad_gx_library:L_Chilisin_MHCI06030, F.Cu at (65.2, 112.2)
- added Q8: AO3400A, Package_TO_SOT_SMD:SOT-23, F.Cu at (133.8, 102.7)
- added Q9: AO3400A, Package_TO_SOT_SMD:SOT-23, F.Cu at (133.8, 107.1)
- added R16: 16.5 2W, Resistor_THT:R_Axial_Power_L20.0mm_W6.4mm_P5.08mm_Vertical, F.Cu at (53.3, 112.4)
- added R7: 24.9 2W, Resistor_THT:R_Axial_Power_L20.0mm_W6.4mm_P5.08mm_Vertical, F.Cu at (53.3, 104.4)
- added U10: LM74610, Package_SO:VSSOP-8_3x3mm_P0.65mm, F.Cu at (127.7, 107.5)
- added U8: LM1085-5.0, Package_TO_SOT_SMD:TO-263-3_TabPin2, F.Cu at (65.7, 122.5)
- added U9: AMS1117-3.3, Package_TO_SOT_SMD:SOT-223-3_TabPin2, F.Cu at (59.9, 132.9)
- BT1, BT2: moved to F.Cu
- C1: value 0.47u/25V -> 0.1u/25V; footprint Capacitor_SMD:C_0805_2012Metric -> Capacitor_SMD:C_0603_1608Metric
- C11: value 10u/25V -> 0.1u/25V; footprint Capacitor_SMD:C_0805_2012Metric -> Capacitor_SMD:C_0603_1608Metric
- C12: value 10u/25V -> 0.47u/25V
- C13, C14: value 22u/16V -> 0.47u/10V; footprint Capacitor_SMD:C_1206_3216Metric -> Capacitor_SMD:C_0603_1608Metric
- C16: value 0.1u/25V -> 0.47u/10V
- C18: value 10u/25V -> 1u/16V
- C19: value 0.1u/25V -> 1u/16V; footprint Capacitor_SMD:C_0603_1608Metric -> Capacitor_SMD:C_0805_2012Metric
- C3, C4, C5: value 0.47u/10V -> 10u/25V; footprint Capacitor_SMD:C_0603_1608Metric -> Capacitor_SMD:C_0805_2012Metric
- C6: value 0.1u/25V -> 10u/25V; footprint Capacitor_SMD:C_0603_1608Metric -> Capacitor_SMD:C_0805_2012Metric
- C7: value 1u/16V -> 0.1u/25V; footprint Capacitor_SMD:C_0805_2012Metric -> Capacitor_SMD:C_0603_1608Metric
- R1, R2: value 150 -> 10k; footprint Resistor_SMD:R_1206_3216Metric -> Resistor_SMD:R_0805_2012Metric
- R10, R9: value 10k -> 150; footprint Resistor_SMD:R_0805_2012Metric -> Resistor_SMD:R_1206_3216Metric
- R11: value 10k -> 0.0025; footprint Resistor_SMD:R_0805_2012Metric -> Resistor_SMD:R_Shunt_Vishay_WSK2512_6332Metric_T2.21mm
- R12: value 10k -> 1k
- R13: value 46.4k -> 820
- R3: value 0.0025 -> 10k; footprint Resistor_SMD:R_Shunt_Vishay_WSK2512_6332Metric_T2.21mm -> Resistor_SMD:R_0805_2012Metric
- R4: value 1k -> 10k
- R5: value 820 -> 68.1k; footprint Resistor_SMD:R_0805_2012Metric -> Resistor_SMD:R_0201_0603Metric
- R6: value 10 -> 46.4k
- R8: value 68.1k -> 10; footprint Resistor_SMD:R_0201_0603Metric -> Resistor_SMD:R_0805_2012Metric
- U1: value ~ -> TPS563201; footprint Package_DFN_QFN:TQFN-24-1EP_4x4mm_P0.5mm_EP2.1x2.1mm -> Package_TO_SOT_SMD:SOT-23-6
- U2: value TPS563201 -> ~; footprint Package_TO_SOT_SMD:SOT-23-6 -> Package_DFN_QFN:TQFN-24-1EP_4x4mm_P0.5mm_EP2.1x2.1mm
- U3: value LM74610 -> TPS563201; footprint Package_SO:VSSOP-8_3x3mm_P0.65mm -> Package_TO_SOT_SMD:SOT-23-6
- U7: value AMS1117-3.3 -> LM74610; footprint Package_TO_SOT_SMD:SOT-223-3_TabPin2 -> Package_SO:VSSOP-8_3x3mm_P0.65mm
- moved C11 165.7 mm to (47.0, 89.7)
- moved C8 163.7 mm to (47.0, 87.2)
- moved C14 151.1 mm to (47.0, 94.7)
- moved C13 150.9 mm to (47.0, 92.2)
- moved R9 145.9 mm to (69.6, 87.6)
- moved R10 145.8 mm to (69.6, 90.9)
- moved JP10 144.2 mm to (47.2, 105.8)
- moved JP9 144.2 mm to (47.2, 102.2)
- moved R8 139.8 mm to (61.0, 87.4)
- moved U2 132.0 mm to (75.6, 88.7)
- moved C12 128.7 mm to (85.3, 91.9)
- moved F2 96.6 mm to (74.5, 94.2)
- moved C18 94.5 mm to (126.2, 111.3)
- moved TP4 89.2 mm to (108.0, 122.2)
- moved BT2 87.8 mm to (48.7, 74.2), turned to 0 degrees
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Connections:
- C1 pad 1: Net-(U1-CP) -> Net-(JP9-B)
- C1 pad 2: Net-(U1-IN) -> GND
- C11 pad 1: Net-(JP2-B) -> Net-(U2-IN)
- C11 pad 2: GND -> GNDREF
- C12 pad 1: Net-(JP2-B) -> Net-(U2-CP)
- C12 pad 2: GND -> Net-(U2-IN)
- C13 pad 1: Net-(JP3-A) -> Net-(U2-REG3)
- C13 pad 2: GND -> GNDREF
- C14 pad 1: Net-(JP3-A) -> Net-(U2-REG2)
- C14 pad 2: GND -> GNDREF
- C16 pad 1: Net-(JP4-B) -> Net-(U2-AOLDO)
- C16 pad 2: GND -> GNDREF
- C18 pad 1: Net-(JP4-B) -> Net-(U7-VCAPH)
- C18 pad 2: GND -> Net-(U7-VCAPL)
- C2 pad 1: Net-(U1-IN) -> Net-(JP10-B)
- C2 pad 2: GNDREF -> GND
- C3 pad 1: Net-(U1-REG3) -> Net-(JP9-B)
- C3 pad 2: GNDREF -> GND
- C4 pad 1: Net-(U1-REG2) -> Net-(JP10-B)
- C4 pad 2: GNDREF -> GND
- C5 pad 1: Net-(U1-AOLDO) -> Net-(JP9-B)
- C5 pad 2: GNDREF -> GND
- C6 pad 1: Net-(U1-CELL1) -> Net-(JP10-B)
- C6 pad 2: GNDREF -> GND
- C7 pad 1: Net-(U3-VCAPH) -> Net-(U1-SW)
- C7 pad 2: Net-(U3-VCAPL) -> Net-(U1-VBST)
- C8 pad 1: Net-(U2-SW) -> Net-(U2-CELL1)
- C8 pad 2: Net-(U2-VBST) -> GNDREF
- JP10 pad 1: Net-(JP10-A) -> /Power Regulation/PWR_IN_SELECT
- JP10 pad 2: VRAW -> Net-(JP10-B)
- JP12 pad 1: Net-(JP1-B) -> Net-(JP12-A)
- JP12 pad 2: +3.3V -> /Battery 18650 Input/PWR_18650
- JP8 pad 2: Net-(JP8-B) -> /Battery_PowerPole_Input/PWR_POWERPOLE
- JP9 pad 1: +7.5V -> /Power Regulation/PWR_IN_SELECT
- Q2 pad 3: +7.5V -> Net-(JP12-A)
- R1 pad 1: Net-(U1-BATTS) -> Net-(JP9-B)
- R1 pad 2: +BATT -> Net-(U1-EN)
- R10 pad 1: Net-(U2-VFB) -> Net-(U2-CELL1)
- R10 pad 2: GND -> Net-(BT1--)
- R11 pad 1: VRAW -> GNDREF
- R11 pad 2: Net-(U6-EN) -> Net-(U2-CSP)
- R12 pad 1: Net-(U6-VFB) -> Net-(JP12-A)
- R12 pad 2: GND -> Net-(U2-PCKP)
- R13 pad 1: Net-(U6-VFB) -> Net-(JP12-A)
- R13 pad 2: Net-(JP5-A) -> Net-(U2-ZVC)
- R2 pad 1: Net-(U1-CELL1) -> Net-(JP10-B)
- R2 pad 2: Net-(BT1--) -> Net-(U3-EN)
- R3 pad 1: GNDREF -> Net-(U1-VFB)
- R3 pad 2: Net-(U1-CSP) -> GND
- R4 pad 1: +7.5V -> Net-(U3-VFB)
- R4 pad 2: Net-(U1-PCKP) -> GND
- R5 pad 1: +7.5V -> Net-(U1-VFB)
- R5 pad 2: Net-(U1-ZVC) -> Net-(JP13-A)
- R6 pad 1: Net-(U1-IN) -> Net-(U3-VFB)
- R6 pad 2: +BATT -> Net-(JP14-A)
- R8 pad 1: Net-(U2-VFB) -> Net-(U2-IN)
- R8 pad 2: Net-(JP3-A) -> +BATT
- R9 pad 1: VRAW -> Net-(U2-BATTS)
- R9 pad 2: Net-(U2-EN) -> +BATT
- TH1 pad 1: Net-(U1-TH1) -> Net-(U2-TH1)
- U1 pad 1: Net-(U1-IN) -> GND
- U1 pad 2: Net-(U1-CP) -> Net-(U1-SW)
- U1 pad 3: Net-(Q2-G1) -> Net-(JP9-B)
- U1 pad 4: Net-(Q2-G2) -> Net-(U1-VFB)
- U1 pad 5: Net-(U1-ZVC) -> Net-(U1-EN)
- U1 pad 6: Net-(U1-PCKP) -> Net-(U1-VBST)
- U2 pad 1: GND -> Net-(U2-IN)
- U2 pad 2: Net-(U2-SW) -> Net-(U2-CP)
- U2 pad 3: Net-(JP2-B) -> Net-(Q2-G1)
- U2 pad 4: Net-(U2-VFB) -> Net-(Q2-G2)
- U2 pad 5: Net-(U2-EN) -> Net-(U2-ZVC)
- U2 pad 6: Net-(U2-VBST) -> Net-(U2-PCKP)
- U3 pad 1: Net-(U3-VCAPL) -> GND
- U3 pad 2: Net-(Q3-G) -> Net-(U3-SW)
- U3 pad 3: unconnected-(U3-NC-Pad3) -> Net-(JP10-B)
- U3 pad 4: Net-(JP9-B) -> Net-(U3-VFB)
- U3 pad 5: unconnected-(U3-NC-Pad5) -> Net-(U3-EN)
- U3 pad 6: Net-(Q3-G) -> Net-(U3-VBST)
- U7 pad 1: GND -> Net-(U7-VCAPL)
- U7 pad 2: Net-(JP1-B) -> Net-(Q8-G)
- U7 pad 3: Net-(JP5-B) -> unconnected-(U7-NC-Pad3)
