File: foxhunt1.kicad_pcb (KiCad board)
At the start: 2 copper layers, 76 parts, among them J3 1377G12-BK, J4 MCV 1,5/ 2-GF-3,81, Q1 AO3400A, Q2 8205A, Q8 AO3400A, Q9 AO3400A, U1 TPS563201, U10 LM74610, U3 TPS563201, U7 LM74610, U8 LM1085-5.0, U9 AMS1117-3.3

Commit message: Re-sync PCB net names and restore netclasses after GUI clobber
Update PCB from Schematic (run natively in KiCad) picked up the net
labels added last commit — jumper-hop nets now carry their real names
on the board (e.g. /Power Regulation/5V_BUCK_VIN instead of
Net-(JP9-B)).

Also restores the three power netclasses and DRC floor overrides,
which got silently wiped: the KiCad GUI had this project open with a
stale in-memory copy of net_settings from before that work existed,
and saved over the on-disk changes when it closed. Recreated and
reassigned all 23 net-to-class mappings against the current
(post-sync) net names, verified via get_netclasses (0 orphan
patterns) before committing.

Co-Authored-By: Claude Sonnet 5 <noreply@anthropic.com>
Connections:
- net Net-(J3-Pin_1) renamed /Battery_PowerPole_Input/12V_RAW
- net Net-(JP10-B) renamed /Power Regulation/3V3_BUCK_VIN
- net Net-(JP12-A) renamed /Battery 18650 Input/BATT_PCKP
- net Net-(JP13-A) renamed /Power Regulation/5V_BUCK_OUT
- net Net-(JP13-B) renamed /Power Regulation/5V_LDO_VIN
- net Net-(JP14-A) renamed /Power Regulation/3V3_BUCK_OUT
- net Net-(JP14-B) renamed /Power Regulation/3V3_LDO_VIN
- net Net-(JP15-B) renamed /Power Regulation/5V_LDO_OUT
- net Net-(JP16-B) renamed /Power Regulation/3V3_LDO_OUT
- net Net-(JP9-B) renamed /Power Regulation/5V_BUCK_VIN
