File: foxhunt1.kicad_sch (KiCad schematic)
At the start: 26 parts, among them Q1 AO3400A, Q2 8205A, Q3 AO3400A, U3 LM74610

Commit message: library rename
Parts:
- F2: footprint gx_lib:PTCC_CLM1612 -> kicad_gx_library:Fuse_PTCC_CLM1612; symbol _gxLib:POLY_FUSE -> kicad_gx_library:POLY_FUSE
- Q2: symbol _gxLib:8205A -> kicad_gx_library:8205A
- U1: symbol _gxLib:MAX17320 -> kicad_gx_library:MAX17320
- U3: symbol _gxLib:LM74610 -> kicad_gx_library:LM74610
Changed lines of the file:
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@@
 	)
 	(symbol
-		(lib_id "_gxLib:POLY_FUSE")
+		(lib_id "kicad_gx_library:POLY_FUSE")
 		(at 82.55 58.42 0)
 		(unit 1)
@@
 			)
 		)
-		(property "Footprint" "gx_lib:PTCC_CLM1612"
+		(property "Footprint" "kicad_gx_library:Fuse_PTCC_CLM1612"
 			(at 82.55 58.42 0)
 			(hide yes)
@@
 	)
 	(symbol
-		(lib_name "LM74610_1")
-		(lib_id "_gxLib:LM74610")
+		(lib_id "kicad_gx_library:LM74610")
 		(at 222.25 67.31 0)
 		(unit 1)
@@
 		(fields_autoplaced yes)
 		(property "Reference" "U3"
-			(at 236.22 88.8298 0)
+			(at 238.76 86.2898 0)
 			(show_name no)
 			(do_not_autoplace no)
@@
 		)
 		(property "Value" "LM74610"
-			(at 222.25 67.31 0)
+			(at 238.76 88.8298 0)
 			(show_name no)
 			(do_not_autoplace no)
@@
 	)
 	(symbol
-		(lib_id "_gxLib:8205A")
+		(lib_id "kicad_gx_library:8205A")
 		(at 114.3 69.85 90)
 		(mirror x)
@@
 	)
 	(symbol
-		(lib_id "_gxLib:MAX17320")
+		(lib_id "kicad_gx_library:MAX17320")
 		(at 104.14 82.55 0)
 		(unit 1)
