File: foxhunt1.kicad_sch (KiCad schematic)
At the start: 26 parts, among them Q1 AO3400A, Q2 8205A, Q3 AO3400A, U3 LM74610

Commit message: Make project library-portable; fix Q2 footprint reference
Vendor the three non-standard libraries (kicad_gx_library,
digikey-kicad-library, SparkFun-KiCad-Libraries) as git submodules
under libs/, and add project-level sym-lib-table/fp-lib-table entries
that resolve them via ${KIPRJMOD}, so the project no longer depends on
this machine's global KiCad library setup.

Also fixes Q2's footprint reference, which pointed at an unregistered
"DigikeyGithub" library nickname left over from a prior library setup;
it now correctly resolves to digikey-kicad-library:SOT23-6L.

Co-Authored-By: Claude Sonnet 5 <noreply@anthropic.com>
Parts:
- Q2: footprint DigikeyGithub:SOT23-6L -> digikey-kicad-library:SOT23-6L
Changed lines of the file:
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@@
 			)
 		)
-		(property "Footprint" "DigikeyGithub:SOT23-6L"
+		(property "Footprint" "digikey-kicad-library:SOT23-6L"
 			(at 114.3 69.85 0)
 			(hide yes)
