File: foxhunt1.kicad_sch (KiCad schematic)
At the start: 26 parts, among them Q1 AO3400A, Q2 8205A, Q3 AO3400A, U3 LM74610

Commit message: hierarchy
Parts:
- removed BT1, BT2: Battery_Cell, Battery:BatteryHolder_MPD_BH-18650-PC, symbol Device:Battery_Cell
- removed C1: 0.47u/25V, Capacitor_SMD:C_0805_2012Metric, symbol Device:C_Small
- removed C2, C6: 0.1u/25V, Capacitor_SMD:C_0603_1608Metric, symbol Device:C_Small
- removed C3, C4, C5: 0.47u/10V, Capacitor_SMD:C_0603_1608Metric, symbol Device:C_Small
- removed C7: 1u/16V, Capacitor_SMD:C_0805_2012Metric, symbol Device:C_Small
- removed F2: CLM1612P1412, kicad_gx_library:Fuse_PTCC_CLM1612, symbol kicad_gx_library:POLY_FUSE
- removed JP10, JP9: SolderJumper_2_Open, Jumper:SolderJumper-2_P1.3mm_Open_TrianglePad1.0x1.5mm, symbol Jumper:SolderJumper_2_Open
- removed Q1, Q3: AO3400A, Package_TO_SOT_SMD:SOT-23, symbol Transistor_FET:AO3400A
- removed Q2: 8205A, digikey-kicad-library:SOT23-6L, symbol kicad_gx_library:8205A
- removed R1, R2: 150, Resistor_SMD:R_1206_3216Metric, symbol PCM_SparkFun-Resistor:R
- removed R3: 0.0025, Resistor_SMD:R_Shunt_Vishay_WSK2512_6332Metric_T2.21mm, symbol Device:R_Shunt_US
- removed R4: 1k, Resistor_SMD:R_0805_2012Metric, symbol PCM_SparkFun-Resistor:R
- removed R5: 820, Resistor_SMD:R_0805_2012Metric, symbol PCM_SparkFun-Resistor:R
- removed R6: 10, Resistor_SMD:R_0805_2012Metric, symbol PCM_SparkFun-Resistor:R
- removed TH1: NCP15XH103F03RC, Resistor_SMD:R_0402_1005Metric, symbol Device:Thermistor_US
- removed TP1, TP2: TestPoint, TestPoint:TestPoint_Pad_D1.5mm, symbol Connector:TestPoint
- removed U1: (no value), Package_DFN_QFN:TQFN-24-1EP_4x4mm_P0.5mm_EP2.1x2.1mm, symbol kicad_gx_library:MAX17320
- removed U3: LM74610, Package_SO:VSSOP-8_3x3mm_P0.65mm, symbol kicad_gx_library:LM74610
Connections:
- no-connect marks 8 -> 0
Other:
- note removed: "X7R 0805"
