File: foxhunt1.kicad_sch (KiCad schematic)
At the start: 0 parts

Commit message: Restore root schematic naming convention, fix stale symbol warnings
Rename power_input.kicad_sch back to foxhunt1.kicad_sch (matching the
project name) so Konnect's project-ownership resolution can find the
root — it doesn't yet support KiCad 10's top_level_sheets feature and
assumes <project>.kicad_sch is always the root. Hierarchy content and
UUIDs are unchanged.

Also runs Update Symbols from Library on battery_18650_input.kicad_sch
and power_regulation.kicad_sch to clear 13 stale lib_symbol_mismatch
ERC warnings (no pins moved). Full hierarchy ERC now passes clean:
0 errors, 0 warnings.

Co-Authored-By: Claude Sonnet 5 <noreply@anthropic.com>
Parts:
- added C18, C19: 1u/16V, Capacitor_SMD:C_0805_2012Metric, symbol Device:C_Small
- added JP20, JP21: SolderJumper_2_Open, Jumper:SolderJumper-2_P1.3mm_Open_TrianglePad1.0x1.5mm, symbol Jumper:SolderJumper_2_Open
- added Q8, Q9: AO3400A, Package_TO_SOT_SMD:SOT-23, symbol Transistor_FET:AO3400A
- added U10, U7: LM74610, Package_SO:VSSOP-8_3x3mm_P0.65mm, symbol kicad_gx_library:LM74610
Connections:
- new net: C18.2, U7.1 (VCAPL)
- new net: Q8.1 (G), U7.2 (GATE_DOWN), U7.6 (GATE_DRIVE)
- new net: C18.1, U7.7 (VCAPH)
- new net: JP20.1 (A), Q8.3 (D), U7.8 (CATHODE)
- new net: C19.1, U10.7 (VCAPH)
- new net: C19.2, U10.1 (VCAPL)
- new net: Q9.1 (G), U10.2 (GATE_DOWN), U10.6 (GATE_DRIVE)
- new net: JP21.1 (A), Q9.3 (D), U10.8 (CATHODE)
- new net Battery 18650 Input/PWR_18650: Q8.2 (S), U7.4 (ANODE)
- new net Battery_PowerPole_Input/PWR_POWERPOLE: Q9.2 (S), U10.4 (ANODE)
- new net Power Regulation/PWR_IN_SELECT: JP20.2 (B), JP21.2 (B)
Other:
- added sheet Battery 18650 Input (battery_18650_input.kicad_sch)
- added sheet Battery_PowerPole_Input (battery_powerpole_input.kicad_sch)
- added sheet Power Regulation (power_regulation.kicad_sch)
- note added: "X7R 0805"
