File: power_regulation.kicad_sch (KiCad schematic)
At the start: 31 parts, among them U2 TPS563201, U5 LM1085-5.0, U6 TPS563201, U7 AMS1117-3.3

Commit message: library rename
Parts:
- removed C15: 22u/16V, Capacitor_SMD:C_1206_3216Metric, symbol Device:C_Small
- added C24: 22u/16V Elec, Capacitor_SMD:C_Elec_5x5.8, symbol Device:C_Small
- added C25: 0.1u/25V, Capacitor_SMD:C_0603_1608Metric, symbol Device:C_Small
- added JP1, JP6: Jumper_2_Open, TestPoint:TestPoint_2Pads_Pitch2.54mm_Drill0.8mm, symbol Jumper:Jumper_2_Open
- added JP11, JP12: SolderJumper_2_Open, Jumper:SolderJumper-2_P1.3mm_Open_TrianglePad1.0x1.5mm, symbol Jumper:SolderJumper_2_Open
- added R14: 16.5 2W, Resistor_THT:R_Axial_Power_L20.0mm_W6.4mm_P5.08mm_Vertical, symbol PCM_SparkFun-Resistor:R
- added R15: 24.9 2W, Resistor_THT:R_Axial_Power_L20.0mm_W6.4mm_P5.08mm_Vertical, symbol PCM_SparkFun-Resistor:R
- L1, L2: footprint gx_lib:L_Chilisin_MHCI06030 -> kicad_gx_library:L_Chilisin_MHCI06030
Connections:
- net +3.3V: now also JP12.2 (B); no longer C22.1, C23.1, U7.2 (VO)
- net +5V: now also JP11.2 (B); no longer U5.2 (VO)
- net GND: now also C24.2, C25.2, R14.1, R15.1
- new net: JP1.1 (A), R14.2
- new net: C22.1, C23.1, JP1.2 (B), JP12.1 (A), U7.2 (VO)
- new net: C24.1, C25.1, JP11.1 (A), JP6.2 (B), U5.2 (VO)
- new net: JP6.1 (A), R15.2
Other:
- note added: "**4.3V**"
- note removed: "**5V**"
- moved on the sheet: C22, C23, U7
