File: power_regulation.kicad_sch (KiCad schematic)
At the start: 38 parts, among them U2 TPS563201, U5 LM1085-5.0, U6 TPS563201, U7 AMS1117-3.3

Commit message: hierarchy
Parts:
- added C32, C33: 0.1u/25V, Capacitor_SMD:C_0603_1608Metric, symbol Device:C_Small
- U8: renamed from U5; LCSC Part # (none) -> C5145336; MPN (none) -> LM1085IS-5.0RG; Manf (none) -> HANSCHIP semiconductor; Package (none) -> TO-263-3L
- renumbered C10 to C1, C19 to C15, C16 to C2, C13 to C28, C20 to C29, C11 to C3, C14 to C30, C21 to C31, C25 to C34, C22 to C35, C24 to C36, C23 to C37, C17 to C4, C12 to C5, C18 to C6, C8 to C7, JP4 to JP10, JP3 to JP13, JP5 to JP14, JP6 to JP15, JP1 to JP16, JP11 to JP17, JP12 to JP18, JP2 to JP9, L1 to L3, L2 to L4, R9 to R1, R14 to R16, R11 to R2, R10 to R3, R12 to R4, R8 to R5, R13 to R6, R15 to R7, U2 to U1, U6 to U3, U7 to U9
Connections:
- net GND: now also C32.2, C33.2
- net at JP14.2 (B), U9.3 (VI): now also C33.1
- net at JP13.2 (B), U8.3 (VI): now also C32.1

Commit message: hierarchy work
Connections:
- net at C1.1, C3.1, C5.1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: now also R1.1
- net at C2.1, C4.1, C6.1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: now also R2.1
- net VRAW renamed PWR_IN_SELECT
- net PWR_IN_SELECT: no longer R1.1, R2.1
Other:
- moved on the sheet: R1, R2
