File: battery_18650_input.kicad_sch (KiCad schematic)
At the start: 0 parts

Commit message: hierarchy work
Parts:
- added BT1, BT2: Battery_Cell, Battery:BatteryHolder_MPD_BH-18650-PC, symbol Device:Battery_Cell
- added C11, C8: 0.1u/25V, Capacitor_SMD:C_0603_1608Metric, symbol Device:C_Small
- added C12: 0.47u/25V, Capacitor_SMD:C_0805_2012Metric, symbol Device:C_Small
- added C13, C14, C16: 0.47u/10V, Capacitor_SMD:C_0603_1608Metric, symbol Device:C_Small
- added F2: CLM1612P1412, kicad_gx_library:Fuse_PTCC_CLM1612, symbol kicad_gx_library:POLY_FUSE
- added JP12: SolderJumper_2_Open, Jumper:SolderJumper-2_P1.3mm_Open_TrianglePad1.0x1.5mm, symbol Jumper:SolderJumper_2_Open
- added Q1: AO3400A, Package_TO_SOT_SMD:SOT-23, symbol Transistor_FET:AO3400A
- added Q2: 8205A, digikey-kicad-library:SOT23-6L, symbol kicad_gx_library:8205A
- added R10, R9: 150, Resistor_SMD:R_1206_3216Metric, symbol PCM_SparkFun-Resistor:R
- added R11: 0.0025, Resistor_SMD:R_Shunt_Vishay_WSK2512_6332Metric_T2.21mm, symbol Device:R_Shunt_US
- added R12: 1k, Resistor_SMD:R_0805_2012Metric, symbol PCM_SparkFun-Resistor:R
- added R13: 820, Resistor_SMD:R_0805_2012Metric, symbol PCM_SparkFun-Resistor:R
- added R8: 10, Resistor_SMD:R_0805_2012Metric, symbol PCM_SparkFun-Resistor:R
- added TH1: NCP15XH103F03RC, Resistor_SMD:R_0402_1005Metric, symbol Device:Thermistor_US
- added TP1, TP2: TestPoint, TestPoint:TestPoint_Pad_D1.5mm, symbol Connector:TestPoint
- added U2: (no value), Package_DFN_QFN:TQFN-24-1EP_4x4mm_P0.5mm_EP2.1x2.1mm, symbol kicad_gx_library:MAX17320
Connections:
- new net: F2.2, Q1.3 (D)
- new net: F2.3, Q2.1 (S1)
- new net: BT1.2 (-), BT2.1 (+), R10.2, TP1.1
- new net: JP12.1 (A), Q2.3 (S2), R12.1, R13.1
- new net: R13.2, U2.5 (ZVC)
- new net: TH1.1, U2.10 (TH1)
- new net: C14.1, U2.17 (REG2)
- new net: C16.1, U2.12 (AOLDO)
- new net: C13.1, U2.13 (REG3)
- new net: C11.1, C12.2, R8.1, U2.1 (IN)
- new net: C12.1, U2.2 (CP)
- new net: R11.2, U2.15 (CSP)
- new net: R11.3, U2.14 (CSN)
- new net: C8.1, R10.1, U2.21 (CELL1), U2.22 (CELL2), U2.23 (CELL3)
- new net: Q1.1 (G), U2.11 (PFAIL)
- new net: R9.1, U2.24 (BATTS)
- new net: Q2.6 (G1), U2.3 (CHG)
- new net: Q2.4 (G2), U2.4 (DIS)
- new net: R12.2, U2.6 (PCKP)
- new net +BATT: BT1.1 (+), F2.1, R8.2, R9.2, TP2.1
- new net GND: R11.4
- new net GNDREF: BT2.2 (-), C11.2, C13.2, C14.2, C16.2, C8.2, Q1.2 (S), R11.1, TH1.2, U2.20 (GND), U2.25 (GND)
- new net PWR_18650: JP12.2 (B)
- no-connect marks 0 -> 8
