File: battery_18650_input.kicad_sch (KiCad schematic)
At the start: 22 parts, among them Q1 AO3400A, Q2 8205A

Commit message: Add project_library, datasheet cross-referencing, and LCSC verification
Task 1: verify every LCSC-sourced component (26 unique parts, 54
instances) against the real JLCPCB catalog. 25 of 26 check out cleanly;
findings and an action-item checklist are in
_docs/task1_lcsc_crossreference.md, including the reclassification that
capacitor voltage ratings are a minimum, not an exact value (not a
defect), with a follow-up task to document that convention on each
sheet.

Task 2: kicad_gx_library's 4 real symbols (LM74610, POLY_FUSE,
MAX17320, 8205A) now have their Datasheet property linked at both the
library-definition and placed-instance level, pointing at local
${KIPRJMOD} paths (submodule commit 62643d1) instead of external URLs.

Task 3: new project_library/ directory holds datasheets for the other
23 unique real parts used in the design (resistors, caps, diode, fuse,
connectors, regulators) with instance-level Datasheet links set the
same way. See _docs/project_library_datasheets.md for the full table
and the handful of parts that couldn't be sourced (BT1/BT2 battery
holder, J3 connector, R16/R7).

Task 4: searched for STEP/IGES 3D models for the custom footprints and
IC packages. Nothing new needed downloading — all 5 standard IC
packages and the Chilisin inductor already resolve to stock KiCad 3D
models, and the Anderson connector already had STEP+IGES on disk.
Two fuse parts remain genuinely gated behind login walls across 8+
sources tried; documented in _docs/3d_models.md with manual-download
links as the practical next step.

Bumps the kicad_gx_library submodule pointer to 62643d1. Also removes
the stray *.pdf .gitignore entry (already unstaged from a prior
session turn) so datasheets in this project can be tracked at all.

Co-Authored-By: Claude Sonnet 5 <noreply@anthropic.com>
Claude-Session: https://claude.ai/code/session_014QW1D2nTw6VPu4FizCgnVk
Parts:
- U2: value (none) -> MAX17320
Changed lines of the file:
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@@
 			)
 		)
-		(property "Datasheet" "https://www.lcsc.com/datasheet/C5353611.pdf"
+		(property "Datasheet" "${KIPRJMOD}/libs/kicad_gx_library/datasheets/Polytronics/CLM1612-12A.pdf"
 			(at 111.76 44.45 0)
 			(hide yes)
@@
 			)
 		)
-		(property "Datasheet" "https://www.lcsc.com/datasheet/C114544.pdf"
+		(property "Datasheet" "${KIPRJMOD}/project_library/datasheets/YAGEO/RC0805FR-07820RL.pdf"
 			(at 191.77 76.2 0)
 			(hide yes)
@@
 			)
 		)
-		(property "Datasheet" "https://www.lcsc.com/datasheet/C77131.pdf"
+		(property "Datasheet" "${KIPRJMOD}/project_library/datasheets/Murata_Electronics/NCP15XH103F03RC.pdf"
 			(at 118.11 116.84 0)
 			(hide yes)
@@
 			)
 		)
-		(property "Datasheet" "https://www.lcsc.com/datasheet/C435402.pdf"
+		(property "Datasheet" "${KIPRJMOD}/project_library/datasheets/Murata_Electronics/GRM188R71A474KA61D.pdf"
 			(at 194.31 97.79 0)
 			(hide yes)
@@
 			)
 		)
-		(property "Datasheet" "https://www.lcsc.com/datasheet/C435402.pdf"
+		(property "Datasheet" "${KIPRJMOD}/project_library/datasheets/Murata_Electronics/GRM188R71A474KA61D.pdf"
 			(at 208.28 97.79 0)
 			(hide yes)
@@
 			)
 		)
-		(property "Datasheet" "https://www.lcsc.com/datasheet/C435402.pdf"
+		(property "Datasheet" "${KIPRJMOD}/project_library/datasheets/Murata_Electronics/GRM188R71A474KA61D.pdf"
 			(at 180.34 97.79 0)
 			(hide yes)
@@
 			)
 		)
-		(property "Datasheet" "https://www.lcsc.com/datasheet/C96347.pdf"
+		(property "Datasheet" "${KIPRJMOD}/project_library/datasheets/YAGEO/RC0805FR-0710RL.pdf"
 			(at 86.36 81.28 0)
 			(hide yes)
@@
 			)
 		)
-		(property "Datasheet" "https://www.lcsc.com/datasheet/C437481.pdf"
+		(property "Datasheet" "${KIPRJMOD}/project_library/datasheets/Murata_Electronics/GCM219R71E474KA55D.pdf"
 			(at 115.57 77.47 0)
 			(hide yes)
@@
 			)
 		)
-		(property "Datasheet" "https://www.lcsc.com/datasheet/C2904234.pdf"
+		(property "Datasheet" "${KIPRJMOD}/project_library/datasheets/Milliohm/HoJLR2512-3W-2.5mR-1_.pdf"
 			(at 152.4 128.27 0)
 			(hide yes)
@@
 			)
 		)
-		(property "Datasheet" "https://www.lcsc.com/datasheet/C77055.pdf"
+		(property "Datasheet" "${KIPRJMOD}/project_library/datasheets/Murata_Electronics/GRM188R71H104KA93D.pdf"
 			(at 102.87 106.68 0)
 			(hide yes)
@@
 			)
 		)
-		(property "Datasheet" "https://www.lcsc.com/datasheet/C20917.pdf"
+		(property "Datasheet" "${KIPRJMOD}/libs/kicad_gx_library/datasheets/Hottech/AO3400.pdf"
 			(at 128.27 66.04 0)
 			(hide yes)
@@
 			)
 		)
-		(property "Value" ""
+		(property "Value" "MAX17320"
 			(at 133.35 68.58 0)
 			(show_name no)
@@
 			)
 		)
-		(property "Datasheet" "https://www.analog.com/media/en/technical-documentation/data-sheets/max17320.pdf"
+		(property "Datasheet" "${KIPRJMOD}/libs/kicad_gx_library/datasheets/Analog_Devices/max17320.pdf"
 			(at 133.35 68.58 0)
 			(hide yes)
@@
 			)
 		)
-		(property "Datasheet" "https://www.lcsc.com/datasheet/C870430.pdf"
+		(property "Datasheet" "${KIPRJMOD}/project_library/datasheets/YAGEO/RT1206BRD07150RL.pdf"
 			(at 86.36 88.9 0)
 			(hide yes)
@@
 			)
 		)
-		(property "Datasheet" "https://www.lcsc.com/datasheet/C870430.pdf"
+		(property "Datasheet" "${KIPRJMOD}/project_library/datasheets/YAGEO/RT1206BRD07150RL.pdf"
 			(at 88.9 106.68 0)
 			(hide yes)
@@
 			)
 		)
-		(property "Datasheet" "https://www.lcsc.com/datasheet/C22458966.pdf"
+		(property "Datasheet" "${KIPRJMOD}/libs/kicad_gx_library/datasheets/JSMICRO/8205A.pdf"
 			(at 143.51 55.88 0)
 			(hide yes)
@@
 			)
 		)
-		(property "Datasheet" "https://www.lcsc.com/datasheet/C95781.pdf"
+		(property "Datasheet" "${KIPRJMOD}/project_library/datasheets/YAGEO/RC0805FR-071KL.pdf"
 			(at 180.34 73.66 0)
 			(hide yes)
@@
 			)
 		)
-		(property "Datasheet" "https://www.lcsc.com/datasheet/C77055.pdf"
+		(property "Datasheet" "${KIPRJMOD}/project_library/datasheets/Murata_Electronics/GRM188R71H104KA93D.pdf"
 			(at 113.03 85.09 0)
 			(hide yes)
