File: battery_powerpole_input.kicad_sch (KiCad schematic)
At the start: 10 parts, among them J3 1377G12-BK, J4 MCV 1,5/ 2-GF-3,81, Q5 AO3400A, U4 LM74610

Commit message: hierarchy work
Parts:
- removed C9: 1u/16V, Capacitor_SMD:C_0805_2012Metric, symbol Device:C_Small
- removed JP7: SolderJumper_2_Open, Jumper:SolderJumper-2_P1.3mm_Open_TrianglePad1.0x1.5mm, symbol Jumper:SolderJumper_2_Open
- removed Q5: AO3400A, Package_TO_SOT_SMD:SOT-23, symbol Transistor_FET:AO3400A
- removed U4: LM74610, Package_SO:VSSOP-8_3x3mm_P0.65mm, symbol kicad_gx_library:LM74610
Connections:
- net PWR_POWERPOLE: now reaches JP8.2 (B)
Other:
- note removed: "X7R 0805"
