File: pcb/battery_powerpole_input.kicad_sch (KiCad schematic)
At the start: 6 parts, among them J3 1377G12-BK, J4 MCV 1,5/ 2-GF-3,81

Commit message: Add ESP32-S3 MCU sheet and CH340C USB-UART programming bridge
Restructures the schematic hierarchy: root sheet now hosts three
top-level sheets (Power, mcu-esp32, USB-C Programming UART) instead of
the old flat layout, with the battery/12V ORing-FET merge circuit
moved into its own dedicated Power sheet. Adds the ESP32-S3-WROOM-1
MCU sheet (native USB-C connector stubbed in but not yet wired) and a
CH340C-based USB-UART bridge with auto-reset/bootloader transistor
circuit for programming.

This is a work-in-progress checkpoint — several nets in the new sheets
(MCU decoupling, CH340C power, auto-reset routing, ORing FET gate
drive) still need wiring before ERC will be clean; see prior review
notes for the punch list.

Co-Authored-By: Claude Sonnet 5 <noreply@anthropic.com>
Claude-Session: https://claude.ai/code/session_01LwTJQ9pyVNMigbu4uLMh8c
Parts:
- renumbered D2 to D1, F3 to F2, J3 to J1, J4 to J2, JP8 to JP4, TP4 to TP3
