File: pcb/battery_powerpole_input.kicad_sch (KiCad schematic)
At the start: 9 parts, among them J2 1377G12-BK, J3 MCV 1,5/ 2-GF-3,81

Commit message: Move audio jack (J6) into SA818V sheet, rename nets/jumpers for clarity
Relocates the switched TRS jack from audio.kicad_sch into SA818V.kicad_sch
and updates the root sheet's pin interface to match (SA818_IN_MIC,
SA818_IN_PTT, new SA818_IN_PTT_HB), fixing an I2C_MIC_OUT/I2S_MIC_OUT
naming typo along the way. Ring/ring-switch/sleeve are wired; tip and
tip-switch (mic audio leg) are still open, per audio_ptt_path.md.

Also: renames GPS hierarchical labels and several power/regulation/
peripheral jumper values from generic (Jumper_2_Open, SolderJumper_2_Open)
to descriptive names, wires MCU_OUT_PTT_HB, and removes now-unused test
points/jumpers from the battery input sheets. Adds 74hc123_pinout.md
planning doc for the TX-safety timeout / force-off failsafe part.

Co-Authored-By: Claude Sonnet 5 <noreply@anthropic.com>
Claude-Session: https://claude.ai/code/session_01P3G1ionr2QCR8SZtKRreL3
Parts:
- removed JP10: Jumper_2_Open, TestPoint:TestPoint_2Pads_Pitch2.54mm_Drill0.8mm, symbol Jumper:Jumper_2_Open
- removed JP11: SolderJumper_2_Open, Jumper:SolderJumper-2_P1.3mm_Open_TrianglePad1.0x1.5mm, symbol Jumper:SolderJumper_2_Open
