File: pcb/battery_powerpole_input.kicad_sch (KiCad schematic)
At the start: 7 parts, among them J2 1377G12-BK, J3 MCV 1,5/ 2-GF-3,81

Commit message: changes on pcb
Parts:
- removed F2: Fuse 2A, kicad_gx_library:Fuse_MCCQ-122, symbol Device:Fuse
- removed TP3: TestPoint, TestPoint:TestPoint_Pad_D1.5mm, symbol Connector:TestPoint
- J3: value MCV 1,5/ 2-GF-3,81 -> 236-102; footprint Connector_Phoenix_MC:PhoenixContact_MCV_1,5_2-GF-3.81_1x02_P3.81mm_Vertical_ThreadedFlange_MountHole -> kicad_gx_library:TerminalBlock_WAGO_236-102_1x02_P5.00mm_45Degree; MPN MCV 1,5/ 2-GF-3,81 -> 236-102; Manf PHOENIX CONTACT -> WAGO Corporation; Mating MPN 1851232 -> (none); Newark PN 69R9760 -> (none); now not fitted
Connections:
- net 12V_RAW is gone; now on net PWR_POWERPOLE: J2.1 (Pin_1), J3.1 (Pin_1)
