File: pcb/foxhunt1.kicad_sch (KiCad schematic)
At the start: 0 parts

Commit message: working through usb-c and hub
Other:
- sheet USB-C Programming UART renamed USB-C
- sheet Power ports: added USB_3.3V_IN, USB_5V_IN; removed none
- sheet USB-C ports: added USB_3.3V, USB_5V, USB_MCU_D+, USB_MCU_D-; removed none
- sheet mcu-esp32 ports: added MCU_USB_D+, MCU_USB_D-; removed none
