File: pcb/mcu-esp32.kicad_sch (KiCad schematic)
At the start: 5 parts, among them J5 HC-TYPE-C-16P-01A, U8 ESP32-S3-WROOM-1-N8R8

Commit message: working through usb-c and hub
Parts:
- removed J5: HC-TYPE-C-16P-01A, Connector_USB:USB_C_Receptacle_HCTL_HC-TYPE-C-16P-01A, symbol Connector:USB_C_Receptacle_USB2.0_16P
- removed R15, R16: 5.1k, Resistor_SMD:R_0603_1608Metric, symbol PCM_SparkFun-Resistor:R
Connections:
- net MCU_USB_D+: now reaches U8.13 (GPIO19/U1RTS/ADC2_CH8/CLK_OUT2/USB_D-)
- net MCU_USB_D-: now reaches U8.14 (GPIO20/U1CTS/ADC2_CH9/CLK_OUT1/USB_D+)
- no-connect marks 6 -> 4
