File: pcb/mcu-esp32.kicad_sch (KiCad schematic)
At the start: 13 parts, among them Q4 BSS138, Q5 BSS138, U10 ESP32-S3-WROOM-1-N8R8

Commit message: annotations
Connections:
- net MCU_ANALOG_RF_DET renamed MCU_OUT_GPS_EXTINT
- net MCU_IN_DIG_RF_DET renamed MCU_IN_EXT_RADIO
Changed lines of the file:
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@@
+	(wire
+		(pts
+			(xy 170.18 80.01) (xy 180.34 80.01)
+		)
+		(stroke
+			(width 0)
+			(type default)
+		)
+	)
 	(wire
 		(pts
@@
 		(pts
 			(xy 227.33 123.19) (xy 227.33 130.81)
-		)
-		(stroke
-			(width 0)
-			(type default)
-		)
-	)
-	(wire
-		(pts
-			(xy 180.34 80.01) (xy 170.18 80.01)
 		)
 		(stroke
@@
 		)
 	)
-	(hierarchical_label "MCU_ANALOG_RF_DET"
-		(shape input)
+	(hierarchical_label "MCU_OUT_GPS_EXTINT"
+		(shape output)
 		(at 180.34 80.01 0)
 		(effects
@@
 		)
 	)
-	(hierarchical_label "MCU_IN_DIG_RF_DET"
+	(hierarchical_label "MCU_IN_EXT_RADIO"
 		(shape input)
 		(at 68.58 74.93 180)
