File: pcb/power.kicad_sch (KiCad schematic)
At the start: 8 parts, among them Q1 AO3400A, Q2 AO3400A, U1 LM74610, U2 LM74610

Commit message: working through usb-c and hub
Other:
- sheet Power Regulation ports: added BATT_3.3V_REG, BATT_5V_REG; removed none
Changed lines of the file:
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@@
+		)
+	)
+	(hierarchical_label "USB_3.3V_IN"
+		(shape input)
+		(at 35.56 166.37 180)
+		(effects
+			(font
+				(size 1.27 1.27)
+			)
+			(justify right)
+		)
+	)
+	(hierarchical_label "USB_5V_IN"
+		(shape input)
+		(at 35.56 163.83 180)
+		(effects
+			(font
+				(size 1.27 1.27)
+			)
+			(justify right)
 		)
 	)
@@
 			)
 		)
+		(pin "BATT_3.3V_REG" output
+			(at 224.79 46.99 180)
+			(effects
+				(font
+					(size 1.27 1.27)
+				)
+				(justify left)
+			)
+		)
+		(pin "BATT_5V_REG" output
+			(at 224.79 49.53 180)
+			(effects
+				(font
+					(size 1.27 1.27)
+				)
+				(justify left)
+			)
+		)
 		(instances
 			(project "foxhunt1"
 				(path "/8399ba4b-9428-480d-8b65-76cf154b97a5/37ac1273-0b70-4a42-ac28-8e382584c4a4"
-					(page "9")
-				)
-			)
+					(page "5")
+				)
+			)
