File: pcb/power.kicad_sch (KiCad schematic)
At the start: 29 parts, among them Q5 AO3407A, SW3 POWER, U1 TPS2121RUXR, U2 TPS2121RUXR, U3 TPS2121RUXR, U4 74LVC1G08

Commit message: fix some drc issues
Connections:
- net MCU_OUT_PWR_LATCH renamed PWR_LATCH
Changed lines of the file:
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@@
-	)
-	(junction
-		(at 200.66 54.61)
-		(diameter 0)
-		(color 0 0 0 0)
 	)
 	(junction
@@
 	(wire
 		(pts
-			(xy 200.66 52.07) (xy 200.66 54.61)
+			(xy 200.66 52.07) (xy 200.66 66.04)
 		)
 		(stroke
@@
 	(wire
 		(pts
-			(xy 204.47 54.61) (xy 200.66 54.61)
-		)
-		(stroke
-			(width 0)
-			(type default)
-		)
-	)
-	(wire
-		(pts
 			(xy 64.77 67.31) (xy 67.31 67.31)
 		)
@@
 		(pts
 			(xy 107.95 55.88) (xy 107.95 58.42)
-		)
-		(stroke
-			(width 0)
-			(type default)
-		)
-	)
-	(wire
-		(pts
-			(xy 200.66 54.61) (xy 200.66 66.04)
 		)
 		(stroke
@@
 		)
 	)
-	(hierarchical_label "MCU_OUT_PWR_LATCH"
+	(hierarchical_label "PWR_LATCH"
 		(shape input)
 		(at 204.47 52.07 0)
 		(effects
 			(font
-				(size 1.27 1.27)
-			)
-			(justify left)
-		)
-	)
-	(hierarchical_label "RTC_PWR_INTERRUPT"
-		(shape input)
-		(at 204.47 54.61 0)
-		(effects
-			(font
