File: pcb/power.kicad_sch (KiCad schematic)
At the start: 33 parts, among them J8 Conn_01x03, Q5 AO3407A, SW3 POWER, U1 TPS2121RUXR, U2 TPS2121RUXR, U3 TPS2121RUXR, U4 74LVC1G08

Commit message: change some 0805s to 0603
Parts:
- R6, R9: footprint Resistor_SMD:R_0805_2012Metric -> Resistor_SMD:R_0603_1608Metric; LCSC Part # C84376 -> C95204; MPN RC0805FR-0710KL -> RT0603BRD0710KL; Package 0805 -> 0603
- renumbered C50 to C4, C42 to C5, D5 to D1, J8 to J1, JP25 to JP5, JP5 to JP6, JP6 to JP7, JP26 to JP8, JP23 to JP9, Q5 to Q1, R29 to R10, R45 to R11, SW3 to SW1
