File: pcb/power.kicad_sch (KiCad schematic)
At the start: 33 parts, among them J1 Conn_01x03, Q1 AO3407A, SW1 POWER, U1 TPS2121RUXR, U2 TPS2121RUXR, U3 TPS2121RUXR, U4 74LVC1G08

Commit message: Move audio jack (J6) into SA818V sheet, rename nets/jumpers for clarity
Relocates the switched TRS jack from audio.kicad_sch into SA818V.kicad_sch
and updates the root sheet's pin interface to match (SA818_IN_MIC,
SA818_IN_PTT, new SA818_IN_PTT_HB), fixing an I2C_MIC_OUT/I2S_MIC_OUT
naming typo along the way. Ring/ring-switch/sleeve are wired; tip and
tip-switch (mic audio leg) are still open, per audio_ptt_path.md.

Also: renames GPS hierarchical labels and several power/regulation/
peripheral jumper values from generic (Jumper_2_Open, SolderJumper_2_Open)
to descriptive names, wires MCU_OUT_PTT_HB, and removes now-unused test
points/jumpers from the battery input sheets. Adds 74hc123_pinout.md
planning doc for the TX-safety timeout / force-off failsafe part.

Co-Authored-By: Claude Sonnet 5 <noreply@anthropic.com>
Claude-Session: https://claude.ai/code/session_01P3G1ionr2QCR8SZtKRreL3
Parts:
- JP1: value Jumper_2_Open -> BATT IN ISO
- JP2: value SolderJumper_2_Open -> BATT IN ISO
- JP3: value Jumper_2_Open -> 12V IN ISO
- JP4: value SolderJumper_2_Open -> 12V IN ISO
- JP5: value Jumper_2_Open -> 5V SEL BYPASS
- JP6: value Jumper_2_Open -> PWR ISO
- JP7: value SolderJumper_2_Open -> PWR ISO
- JP8: value Jumper_2_Open -> 3.3V SEL BYPASS
- JP9: value Jumper_2_Open -> MAIN SW BYPASS
Changed lines of the file:
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@@
 			)
 		)
-		(property "Value" "SolderJumper_2_Open"
+		(property "Value" "BATT IN ISO"
 			(at 71.12 30.48 0)
 			(show_name no)
@@
 			)
 		)
-		(property "Value" "Jumper_2_Open"
+		(property "Value" "BATT IN ISO"
 			(at 71.12 21.59 0)
+			(hide yes)
 			(show_name no)
 			(do_not_autoplace no)
@@
 			)
 		)
-		(property "Value" "Jumper_2_Open"
+		(property "Value" "PWR ISO"
 			(at 113.03 85.09 0)
+			(hide yes)
 			(show_name no)
 			(do_not_autoplace no)
@@
 			)
 		)
-		(property "Value" "SolderJumper_2_Open"
+		(property "Value" "12V IN ISO"
 			(at 72.39 63.5 0)
 			(show_name no)
@@
 			)
 		)
-		(property "Value" "SolderJumper_2_Open"
+		(property "Value" "PWR ISO"
 			(at 113.03 93.98 0)
 			(show_name no)
@@
 			)
 		)
-		(property "Value" "Jumper_2_Open"
+		(property "Value" "12V IN ISO"
 			(at 72.39 54.61 0)
+			(hide yes)
 			(show_name no)
 			(do_not_autoplace no)
@@
 			)
 		)
-		(property "Value" "Jumper_2_Open"
+		(property "Value" "3.3V SEL BYPASS"
 			(at 123.19 104.14 0)
 			(show_name no)
@@
 			)
 		)
-		(property "Value" "Jumper_2_Open"
+		(property "Value" "MAIN SW BYPASS"
 			(at 213.36 81.28 0)
 			(show_name no)
@@
 			)
 		)
-		(property "Value" "Jumper_2_Open"
+		(property "Value" "5V SEL BYPASS"
 			(at 105.41 152.654 0)
 			(show_name no)
