File: pcb/power_regulation.kicad_sch (KiCad schematic)
At the start: 40 parts, among them U4 TPS563201, U5 TPS563201, U6 LM1085-5.0, U7 AMS1117-3.3

Commit message: working through usb-c and hub
Connections:
- net +3.3V renamed BATT_3.3V_REG
- net +5V renamed BATT_5V_REG
Changed lines of the file:
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@@
 	)
 	(junction
-		(at 276.86 138.43)
-		(diameter 0)
-		(color 0 0 0 0)
-	)
-	(junction
 		(at 231.14 138.43)
 		(diameter 0)
@@
 	)
 	(junction
-		(at 55.88 143.51)
+		(at 269.24 60.96)
 		(diameter 0)
 		(color 0 0 0 0)
 	)
 	(junction
-		(at 269.24 60.96)
+		(at 55.88 143.51)
 		(diameter 0)
 		(color 0 0 0 0)
@@
 	)
 	(junction
+		(at 276.86 138.43)
+		(diameter 0)
+		(color 0 0 0 0)
+	)
+	(junction
 		(at 149.86 138.43)
 		(diameter 0)
@@
 	(wire
 		(pts
+			(xy 276.86 128.27) (xy 276.86 138.43)
+		)
+		(stroke
+			(width 0)
+			(type default)
+		)
+	)
+	(wire
+		(pts
 			(xy 55.88 152.4) (xy 55.88 156.21)
 		)
@@
 	(wire
 		(pts
+			(xy 269.24 53.34) (xy 269.24 60.96)
+		)
+		(stroke
+			(width 0)
+			(type default)
+		)
+	)
+	(wire
+		(pts
 			(xy 114.3 138.43) (xy 134.62 138.43)
 		)
@@
 	(wire
 		(pts
+			(xy 266.7 128.27) (xy 276.86 128.27)
+		)
+		(stroke
+			(width 0)
+			(type default)
+		)
+	)
+	(wire
+		(pts
 			(xy 149.86 138.43) (xy 165.1 138.43)
 		)
@@
 	(wire
 		(pts
+			(xy 270.51 53.34) (xy 269.24 53.34)
+		)
+		(stroke
+			(width 0)
+			(type default)
+		)
+	)
+	(wire
+		(pts
 			(xy 100.33 68.58) (xy 113.03 68.58)
 		)
@@
 	(wire
 		(pts
-			(xy 13.97 85.09) (xy 13.97 88.9)
+			(xy 269.24 124.46) (xy 266.7 124.46)
 		)
 		(stroke
@@
 	(wire
 		(pts
-			(xy 247.65 78.74) (xy 250.19 78.74)
+			(xy 13.97 85.09) (xy 13.97 88.9)
 		)
 		(stroke
@@
 	(wire
 		(pts
-			(xy 218.44 140.97) (xy 218.44 138.43)
+			(xy 247.65 78.74) (xy 250.19 78.74)
 		)
 		(stroke
@@
 	(wire
 		(pts
-			(xy 20.32 66.04) (xy 24.13 66.04)
+			(xy 218.44 140.97) (xy 218.44 138.43)
 		)
 		(stroke
@@
 	(wire
 		(pts
-			(xy 269.24 58.42) (xy 269.24 60.96)
+			(xy 20.32 66.04) (xy 24.13 66.04)
 		)
 		(stroke
@@
 	(wire
 		(pts
-			(xy 276.86 138.43) (xy 276.86 134.62)
+			(xy 266.7 124.46) (xy 266.7 128.27)
 		)
 		(stroke
@@
 		)
 	)
+	(hierarchical_label "BATT_3.3V_REG"
+		(shape output)
+		(at 269.24 124.46 0)
+		(effects
+			(font
+				(size 1.27 1.27)
+			)
+			(justify left)
+		)
+	)
 	(hierarchical_label "PWR_IN_SELECT"
 		(shape input)
@@
 		)
 	)
+	(hierarchical_label "BATT_5V_REG"
+		(shape output)
+		(at 270.51 53.34 0)
+		(effects
+			(font
+				(size 1.27 1.27)
+			)
+			(justify left)
+		)
+	)
 	(symbol
 		(lib_id "PCM_SparkFun-Resistor:R")
@@
 	)
 	(symbol
-		(lib_id "power:+5V")
-		(at 269.24 58.42 0)
-		(unit 1)
-		(body_style 1)
-		(exclude_from_sim no)
-		(in_bom yes)
-		(on_board yes)
-		(in_pos_files yes)
-		(dnp no)
-		(fields_autoplaced yes)
-		(property "Reference" "#PWR035"
-			(at 269.24 62.23 0)
-			(hide yes)
-			(show_name no)
-			(do_not_autoplace no)
-			(effects
-				(font
-					(size 1.27 1.27)
-				)
-			)
-		)
-		(property "Value" "+5V"
-			(at 269.24 53.34 0)
-			(show_name no)
-			(do_not_autoplace no)
-			(effects
-				(font
-					(size 1.27 1.27)
-				)
-			)
-		)
-		(property "Footprint" ""
-			(at 269.24 58.42 0)
-			(hide yes)
-			(show_name no)
-			(do_not_autoplace no)
-			(effects
-				(font
-					(size 1.27 1.27)
-				)
-			)
-		)
-		(property "Datasheet" ""
-			(at 269.24 58.42 0)
-			(hide yes)
-			(show_name no)
-			(do_not_autoplace no)
-			(effects
-				(font
-					(size 1.27 1.27)
-				)
-			)
-		)
-		(property "Description" "Power symbol creates a global label with name \"+5V\""
-			(at 269.24 58.42 0)
-			(hide yes)
-			(show_name no)
-			(do_not_autoplace no)
-			(effects
-				(font
-					(size 1.27 1.27)
-				)
-			)
-		)
-		(pin "1"
-		)
-		(instances
-			(project "foxhunt1"
-				(path "/8399ba4b-9428-480d-8b65-76cf154b97a5/37ac1273-0b70-4a42-ac28-8e382584c4a4/c018545d-e009-44ea-af7b-4949ceaf3d2e"
-					(reference "#PWR035")
-					(unit 1)
-				)
-			)
-		)
-	)
-	(symbol
 		(lib_id "PCM_SparkFun-Resistor:R")
 		(at 106.68 76.2 90)
@@
 					(unit 1)
 				)
-			)
-		)
-	)
-	(symbol
-		(lib_id "power:+3.3V")
-		(at 276.86 134.62 0)
-		(unit 1)
-		(body_style 1)
-		(exclude_from_sim no)
-		(in_bom yes)
-		(on_board yes)
-		(in_pos_files yes)
-		(dnp no)
-		(fields_autoplaced yes)
-		(property "Reference" "#PWR036"
-			(at 276.86 138.43 0)
-			(hide yes)
-			(show_name no)
-			(do_not_autoplace no)
-			(effects
-				(font
-					(size 1.27 1.27)
-				)
-			)
-		)
-		(property "Value" "+3.3V"
-			(at 276.86 129.54 0)
-			(show_name no)
-			(do_not_autoplace no)
-			(effects
-				(font
-					(size 1.27 1.27)
-				)
-			)
-		)
-		(property "Footprint" ""
-			(at 276.86 134.62 0)
-			(hide yes)
-			(show_name no)
-			(do_not_autoplace no)
-			(effects
-				(font
-					(size 1.27 1.27)
-				)
-			)
-		)
-		(property "Datasheet" ""
-			(at 276.86 134.62 0)
-			(hide yes)
-			(show_name no)
-			(do_not_autoplace no)
-			(effects
-				(font
-					(size 1.27 1.27)
-				)
-			)
-		)
-		(property "Description" "Power symbol creates a global label with name \"+3.3V\""
-			(at 276.86 134.62 0)
-			(hide yes)
-			(show_name no)
-			(do_not_autoplace no)
-			(effects
-				(font
-					(size 1.27 1.27)
-				)
-			)
-		)
-		(pin "1"
-		)
-		(instances
-			(project "foxhunt1"
-				(path "/8399ba4b-9428-480d-8b65-76cf154b97a5/37ac1273-0b70-4a42-ac28-8e382584c4a4/c018545d-e009-44ea-af7b-4949ceaf3d2e"
-					(reference "#PWR036")
-					(unit 1)
-				)
