File: pcb/power_regulation.kicad_sch (KiCad schematic)
At the start: 46 parts, among them U6 TPS563201, U7 TPS563201, U8 LM1085-5.0, U9 AMS1117-3.3

Commit message: Wire up PCA9555 expansion IO section, source LEDs/resistors, swap 3.3V LDO to LM1117
- PCA9555PW expansion IO: DIP switch (SW4, IO0_0-3), onboard buttons
  (SW7-10), status LEDs (D7-10) with sourced series resistors, external
  JST breakouts (J4-7/R39-42) for IO0_4-7, INT pull-up (R34), VDD bypass
  (C49), address pins grounded (addr 0x20)
- Route PCA9555 INT (PERIPH_IO_INT) across the Power/mcu-esp32 top-level
  sheets to the ESP32-S3 (MCU_IN_IO_INT)
- Source real YAGEO MPN/LCSC part numbers for R30/R31/R34-R42
- Fix D10 LED (was orange 0603 with an LCSC part# that resolved to a
  different, wrong part) -> yellow 0805 APTD2012LSYCK, verified Vf/LCSC
  match, matching D7-9's package family
- Fix stale copy-pasted Datasheet links on D7-9 and R31/R35
- Swap 3.3V LDO from AMS1117-3.3 to TI LM1117IMPX-3.3/NOPB (5V LDO swap
  from LM1085IS-5.0 still pending)

Co-Authored-By: Claude Sonnet 5 <noreply@anthropic.com>
Claude-Session: https://claude.ai/code/session_01LhLkuH6sQ5GbUZ61bG7p2h
Parts:
- U8: LCSC Part # C5145336 -> C2865978; Manf HANSCHIP semiconductor -> TI; Package TO-263-3L -> DDPAK-3(TO-263-3)
- U9: value AMS1117-3.3 -> LM1117IMPX-3.3; footprint Package_TO_SOT_SMD:SOT-223-3_TabPin2 -> Package_TO_SOT_SMD:SOT-223; symbol Regulator_Linear:AMS1117-3.3 -> PCM_SparkFun-Regulator:LM1117-3.3; IMax (none) -> 800mA; LCSC Part # C6186 -> C23984; MPN AMS1117-3.3 -> LM1117IMPX-3.3/NOPB; Manf Advanced Monolithic Systems -> TI; VMax (none) -> 15V
Changed lines of the file:
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@@
 	)
 	(symbol
-		(lib_id "Regulator_Linear:AMS1117-3.3")
+		(lib_id "PCM_SparkFun-Regulator:LM1117-3.3")
 		(at 208.28 138.43 0)
 		(unit 1)
@@
 		(fields_autoplaced yes)
 		(property "Reference" "U9"
-			(at 208.28 132.08 0)
-			(show_name no)
-			(do_not_autoplace no)
-			(effects
-				(font
-					(size 1.27 1.27)
-				)
-			)
-		)
-		(property "Value" "AMS1117-3.3"
-			(at 208.28 134.62 0)
-			(show_name no)
-			(do_not_autoplace no)
-			(effects
-				(font
-					(size 1.27 1.27)
-				)
-			)
-		)
-		(property "Footprint" "Package_TO_SOT_SMD:SOT-223-3_TabPin2"
-			(at 208.28 133.35 0)
-			(hide yes)
-			(show_name no)
-			(do_not_autoplace no)
-			(effects
-				(font
-					(size 1.27 1.27)
-				)
-			)
-		)
-		(property "Datasheet" "${KIPRJMOD}/project_library/datasheets/Advanced_Monolithic_Systems/AMS1117-3.3.pdf"
-			(at 210.82 144.78 0)
-			(hide yes)
-			(show_name no)
-			(do_not_autoplace no)
-			(effects
-				(font
-					(size 1.27 1.27)
-				)
-			)
-		)
-		(property "Description" "1A Low Dropout regulator, positive, 3.3V fixed output, SOT-223"
+			(at 208.28 127 0)
+			(show_name no)
+			(do_not_autoplace no)
+			(effects
+				(font
+					(size 1.27 1.27)
+				)
+			)
+		)
+		(property "Value" "LM1117IMPX-3.3"
+			(at 208.28 129.54 0)
+			(show_name no)
+			(do_not_autoplace no)
+			(effects
+				(font
+					(size 1.27 1.27)
+				)
+			)
+		)
+		(property "Footprint" "Package_TO_SOT_SMD:SOT-223"
+			(at 208.28 158.75 0)
+			(hide yes)
+			(show_name no)
+			(do_not_autoplace no)
+			(effects
+				(font
+					(size 1.27 1.27)
+				)
+			)
+		)
+		(property "Datasheet" "https://www.lcsc.com/datasheet/C23984.pdf"
+			(at 208.28 153.67 0)
+			(hide yes)
+			(show_name no)
+			(do_not_autoplace no)
+			(effects
+				(font
+					(size 1.27 1.27)
+				)
+			)
+		)
+		(property "Description" "800-mA Low-Dropout Linear Regulator"
+			(at 208.28 156.21 0)
+			(hide yes)
+			(show_name no)
+			(do_not_autoplace no)
+			(effects
+				(font
+					(size 1.27 1.27)
+				)
+			)
+		)
+		(property "MPN" "LM1117IMPX-3.3/NOPB"
 			(at 208.28 138.43 0)
 			(hide yes)
@@
 			)
 		)
-		(property "MPN" "AMS1117-3.3"
+		(property "Manf" "TI"
 			(at 208.28 138.43 0)
 			(hide yes)
@@
 			)
 		)
-		(property "Manf" "Advanced Monolithic Systems"
-			(at 208.28 138.43 0)
-			(hide yes)
-			(show_name no)
-			(do_not_autoplace no)
-			(effects
-				(font
-					(size 1.27 1.27)
-				)
-			)
-		)
-		(property "LCSC Part #" "C6186"
+		(property "LCSC Part #" "C23984"
 			(at 208.28 138.43 0)
 			(hide yes)
@@
 			(at 208.28 138.43 0)
 			(hide yes)
+			(show_name no)
+			(do_not_autoplace no)
+			(effects
+				(font
+					(size 1.27 1.27)
+				)
+			)
+		)
+		(property "VMax" "15V"
+			(at 208.28 132.08 0)
+			(show_name no)
+			(do_not_autoplace no)
+			(effects
+				(font
+					(size 1.27 1.27)
+				)
+			)
+		)
+		(property "IMax" "800mA"
+			(at 208.28 134.62 0)
 			(show_name no)
 			(do_not_autoplace no)
@@
 			)
 		)
-		(property "Datasheet" "${KIPRJMOD}/project_library/datasheets/HANSCHIP_semiconductor/LM1085IS-5.0RG.pdf"
+		(property "Datasheet" "https://www.ti.com/cn/lit/ds/symlink/lm1084.pdf"
 			(at 205.74 60.96 0)
 			(hide yes)
@@
 			)
 		)
-		(property "Description" "3A 25V Linear Regulator, Fixed Output 5.0V, TO-220/TO-263"
+		(property "Description" "5.5A, 29V linear regulator"
 			(at 205.74 60.96 0)
 			(hide yes)
@@
 			)
 		)
-		(property "Manf" "HANSCHIP semiconductor"
+		(property "Manf" "TI"
 			(at 205.74 60.96 0)
 			(hide yes)
@@
 			)
 		)
-		(property "LCSC Part #" "C5145336"
+		(property "LCSC Part #" "C2865978"
 			(at 205.74 60.96 0)
 			(hide yes)
@@
 			)
 		)
-		(property "Package" "TO-263-3L"
+		(property "Package" "DDPAK-3(TO-263-3)"
 			(at 205.74 60.96 0)
 			(hide yes)

Commit message: Wire SD card interface, fix R29/Q6/Q7 sourcing, localize datasheets project-wide
- SD card (Card1, Molex 472192001) wired to the FSPI (SPI2) peripheral:
  IO10/FSPICS0->CS, IO11/FSPID->MOSI, IO12/FSPICLK->SCLK, IO13/FSPIQ->MISO;
  shield/mounting tabs renamed SHLD and grounded; local decoupling cap added
- R29 was silently a 10k YAGEO part (RC0603FR-0710KL/C98220) sitting under a
  1M designator -- corrected to the real 1M part (RC0603FR-071ML/C105578),
  matching this rail's documented VRAW soft-latch bleed design intent
- Q6, Q7 (BSS138): added missing Manf/MPN/LCSC Part# (onsemi BSS138LT1G,
  C82045)
- C32/C36: normalized Value strings; fixed C36's Datasheet, which pointed to
  a different capacitor's PDF entirely
- Localized every remaining component's Datasheet field to a project-local
  path across all 8 schematic sheets (was a live remote URL before), per
  the new datasheet-localization task; caught and rejected a wrong-language
  and a wrong-manufacturer-clone source along the way (U8, U14, U15, Y2)
- Fixed 4 datasheet fields (Q1, D1, U6, U7) that had reverted from their
  already-localized paths back to remote URLs, apparently from a native
  KiCad symbol-library resync picking up stale library-level defaults

Co-Authored-By: Claude Sonnet 5 <noreply@anthropic.com>
Claude-Session: https://claude.ai/code/session_01LhLkuH6sQ5GbUZ61bG7p2h
Parts:
- U9: footprint Package_TO_SOT_SMD:SOT-223 -> PCM_SparkFun-Semiconductor-Standard:SOT-223-3_TabPin2; PROD_ID (none) -> IC-26292
Changed lines of the file:
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@@
 			)
 		)
-		(property "Description" "CAP CER 22uF 16V X7R 1206"
+		(property "Description" "Unpolarized capacitor, small symbol"
 			(at 149.86 153.67 0)
 			(hide yes)
@@
 			)
 		)
-		(property "Description" "RES 10kΩ ±0.1% 100mW 0603"
+		(property "Description" "Resistor, US symbol"
 			(at 107.95 153.67 0)
 			(hide yes)
@@
 			)
 		)
-		(property "Description" "RES 76.8kΩ ±0.1% 100mW 0603"
+		(property "Description" "Resistor, US symbol"
 			(at 121.92 71.12 0)
 			(hide yes)
@@
 			)
 		)
-		(property "Description" "CAP CER 100nF 50V X7R 0603"
+		(property "Description" "Unpolarized capacitor, small symbol"
 			(at 218.44 153.67 0)
 			(hide yes)
@@
 			)
 		)
-		(property "Description" "CAP CER 22uF 16V X7R 1206"
+		(property "Description" "Unpolarized capacitor, small symbol"
 			(at 165.1 153.67 0)
 			(hide yes)
@@
 			)
 		)
-		(property "Description" "CAP CER 100nF 50V X7R 0603"
+		(property "Description" "Unpolarized capacitor, small symbol"
 			(at 113.03 74.93 0)
 			(hide yes)
@@
 			)
 		)
-		(property "Description" "RES 10kΩ ±0.1% 100mW 0603"
+		(property "Description" "Resistor, US symbol"
 			(at 106.68 76.2 0)
 			(hide yes)
@@
 			)
 		)
-		(property "Footprint" "Package_TO_SOT_SMD:SOT-223"
+		(property "Footprint" "PCM_SparkFun-Semiconductor-Standard:SOT-223-3_TabPin2"
 			(at 208.28 158.75 0)
 			(hide yes)
@@
 			)
 		)
-		(property "Datasheet" "https://www.lcsc.com/datasheet/C23984.pdf"
+		(property "Datasheet" "http://www.ti.com/lit/ds/symlink/lm1117.pdf"
 			(at 208.28 153.67 0)
 			(hide yes)
@@
 			)
 		)
-		(property "Description" "800-mA Low-Dropout Linear Regulator"
+		(property "Description" "800mA Low-Dropout Linear Regulator, 3.3V fixed output, SOT-223"
 			(at 208.28 156.21 0)
 			(hide yes)
@@
 			)
 		)
+		(property "PROD_ID" "IC-26292"
+			(at 208.28 161.29 0)
+			(hide yes)
+			(show_name no)
+			(do_not_autoplace no)
+			(effects
+				(font
+					(size 1.27 1.27)
+				)
+			)
+		)
 		(pin "2"
 		)
@@
 			)
 		)
-		(property "Description" "CAP CER 100nF 50V X7R 0603"
+		(property "Description" "Unpolarized capacitor, small symbol"
 			(at 38.1 82.55 0)
 			(hide yes)
@@
 			)
 		)
-		(property "Description" "CAP CER 100nF 50V X7R 0603"
+		(property "Description" "Unpolarized capacitor, small symbol"
 			(at 231.14 153.67 0)
 			(hide yes)
@@
 			)
 		)
-		(property "Description" "CAP CER 10uF 25V X7R 0805"
+		(property "Description" "Unpolarized capacitor, small symbol"
 			(at 67.31 82.55 0)
 			(hide yes)
@@
 			)
 		)
-		(property "Description" "FIXED IND 3.3uH 6A 35mΩ SMD,7.3x6.6mm"
+		(property "Description" "Inductor"
 			(at 138.43 138.43 0)
 			(hide yes)
@@
 			)
 		)
-		(property "Description" "CAP CER 100nF 50V X7R 0603"
+		(property "Description" "Unpolarized capacitor, small symbol"
 			(at 214.63 76.2 0)
 			(hide yes)
@@
 			)
 		)
-		(property "Description" "CAP CER 100nF 50V X7R 0603"
+		(property "Description" "Unpolarized capacitor, small symbol"
 			(at 194.31 153.67 0)
 			(hide yes)
@@
 			)
 		)
-		(property "Description" "CAP CER 100nF 50V X7R 0603"
+		(property "Description" "Unpolarized capacitor, small symbol"
 			(at 39.37 160.02 0)
 			(hide yes)
@@
 			)
 		)
-		(property "Datasheet" "https://www.ti.com/cn/lit/ds/symlink/lm1084.pdf"
+		(property "Datasheet" "http://www.ti.com/lit/ds/symlink/lm1085.pdf"
 			(at 205.74 60.96 0)
 			(hide yes)
@@
 			)
 		)
-		(property "Description" "5.5A, 29V linear regulator"
+		(property "Description" "3A 25V Linear Regulator, Fixed Output 5.0V, TO-220/TO-263"
 			(at 205.74 60.96 0)
 			(hide yes)
@@
 			)
 		)
-		(property "Description" "CAP CER 100nF 50V X7R 0603"
+		(property "Description" "Unpolarized capacitor, small symbol"
 			(at 114.3 152.4 0)
 			(hide yes)
@@
 			)
 		)
-		(property "Description" "CAP CER 100nF 50V X7R 0603"
+		(property "Description" "Unpolarized capacitor, small symbol"
 			(at 193.04 78.74 0)
 			(hide yes)
@@
 			)
 		)
-		(property "Description" "FIXED IND 3.3uH 6A 35mΩ SMD,7.3x6.6mm"
+		(property "Description" "Inductor"
 			(at 137.16 60.96 0)
 			(hide yes)
@@
 			)
 		)
-		(property "Description" "CAP CER 10uF 25V X7R 0805"
+		(property "Description" "Unpolarized capacitor, small symbol"
 			(at 55.88 160.02 0)
 			(hide yes)
@@
 			)
 		)
-		(property "Description" "RES 52.3kΩ ±0.1% 100mW 0603"
+		(property "Description" "Resistor, US symbol"
 			(at 123.19 148.59 0)
 			(hide yes)
@@
 			)
 		)
-		(property "Description" "CAP CER 100nF 50V X7R 0603"
+		(property "Description" "Unpolarized capacitor, small symbol"
 			(at 228.6 76.2 0)
 			(hide yes)
@@
 			)
 		)
-		(property "Description" "CAP CER 22uF 16V X7R 1206"
+		(property "Description" "Unpolarized capacitor, small symbol"
 			(at 163.83 76.2 0)
 			(hide yes)
@@
 			)
 		)
-		(property "Description" "CAP CER 10uF 25V X7R 0805"
+		(property "Description" "Unpolarized capacitor, small symbol"
 			(at 68.58 160.02 0)
 			(hide yes)
@@
 			)
 		)
-		(property "Description" "CAP CER 10uF 25V X7R 0805"
+		(property "Description" "Unpolarized capacitor, small symbol"
 			(at 54.61 82.55 0)
 			(hide yes)
@@
 			)
 		)
-		(property "Description" "CAP CER 22uF 16V X7R 1206"
+		(property "Description" "Unpolarized capacitor, small symbol"
 			(at 148.59 76.2 0)
 			(hide yes)

Commit message: Fix remaining mass-symbol-update reversions (67 Datasheet + 5 Footprint fields)
The project-wide "Update Symbols from Library" run reverted far more than
the 4 caught in the previous commit -- most of that commit's own claimed
"localized project-wide" state was actually already the reverted state,
since the mass update happened before that commit and git history alone
couldn't detect it. Cross-referenced every component's Datasheet/Footprint
against the independent tracking docs (project_library_datasheets.md,
kicad_gx_library_datasheets.md, footprint_verification_log.md) instead.

- 67 components: Datasheet reverted from a localized ${KIPRJMOD} path back
  to a remote URL, across all 8 schematic files
- 5 components: Footprint also reverted, not just Datasheet -- Y2 (RTC
  crystal) reverted to a physically different package size (5.0x3.2mm vs.
  the real 3.2x1.5mm part); U9/U12 (LM1117 LDOs), U10 (ESP32-S3 module),
  and Y1 (12MHz crystal) reverted to differently-sourced but plausible
  footprints from a vendored library instead of the verified stock ones

No MPN/Manf/LCSC Part#/Value regressions found (checked all 185
components). ERC clean, same 15 pre-existing errors as before.

Co-Authored-By: Claude Sonnet 5 <noreply@anthropic.com>
Claude-Session: https://claude.ai/code/session_01LhLkuH6sQ5GbUZ61bG7p2h
Parts:
- U9: footprint PCM_SparkFun-Semiconductor-Standard:SOT-223-3_TabPin2 -> Package_TO_SOT_SMD:SOT-223
Changed lines of the file:
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@@
 			)
 		)
-		(property "Datasheet" "${KIPRJMOD}/project_library/datasheets/YAGEO/RC0805FR-0710KL.pdf"
+		(property "Datasheet" "${KIPRJMOD}/project_library/datasheets/YAGEO/RT0603BRD0710KL.pdf"
 			(at 106.68 76.2 0)
 			(hide yes)
@@
 			)
 		)
-		(property "Footprint" "PCM_SparkFun-Semiconductor-Standard:SOT-223-3_TabPin2"
+		(property "Footprint" "Package_TO_SOT_SMD:SOT-223"
 			(at 208.28 158.75 0)
 			(hide yes)
@@
 			)
 		)
-		(property "Datasheet" "http://www.ti.com/lit/ds/symlink/lm1117.pdf"
+		(property "Datasheet" "${KIPRJMOD}/project_library/datasheets/TI/LM1117IMPX-3.3_NOPB.pdf"
 			(at 208.28 153.67 0)
 			(hide yes)
@@
 			)
 		)
-		(property "Datasheet" "http://www.ti.com/lit/ds/symlink/lm1085.pdf"
+		(property "Datasheet" "${KIPRJMOD}/project_library/datasheets/TI/LM1085IS-5.0RG.pdf"
 			(at 205.74 60.96 0)
 			(hide yes)
