File: pcb/power_regulation.kicad_sch (KiCad schematic)
At the start: 46 parts, among them U6 TPS563201, U7 TPS563201, U8 LM1085-5.0, U9 LM1117IMPX-3.3

Commit message: change some 0805s to 0603
Parts:
- removed C12, C13: 0.1u/25V, Capacitor_SMD:C_0603_1608Metric, symbol Device:C_Small
- removed C16: 10u/25V, Capacitor_SMD:C_0805_2012Metric, symbol Device:C_Small
- removed R16, R17: 10k, Resistor_SMD:R_0805_2012Metric, symbol Device:R_US
- added C14: 0.1u/25V, Capacitor_SMD:C_0603_1608Metric, symbol Device:C_Small
- added C18, C19: 10u/25V, Capacitor_SMD:C_0603_1608Metric, symbol Device:C_Small
- added R18, R19: 10k, Resistor_SMD:R_0603_1608Metric, symbol Device:R_US
- C15: value 10u/25V -> 0.1u/25V; footprint Capacitor_SMD:C_0805_2012Metric -> Capacitor_SMD:C_0603_1608Metric; LCSC Part # C237493 -> C77055; MPN GRM21BZ71E106KE15L -> GRM188R71H104KA93D; Package 0805 -> 0603
- C16: renamed from C14; footprint Capacitor_SMD:C_0805_2012Metric -> Capacitor_SMD:C_0603_1608Metric; LCSC Part # C237493 -> C344022; MPN GRM21BZ71E106KE15L -> GRM188R61E106KA73D
- C17: footprint Capacitor_SMD:C_0805_2012Metric -> Capacitor_SMD:C_0603_1608Metric; LCSC Part # C237493 -> C344022; MPN GRM21BZ71E106KE15L -> GRM188R61E106KA73D
- renumbered C18 to C20, C19 to C21, C20 to C22, C21 to C23, C22 to C24, C23 to C25, C24 to C26, C25 to C27, C26 to C28, C27 to C29, C28 to C30, C29 to C31, JP9 to JP12, JP10 to JP13, JP11 to JP14, JP12 to JP15, JP13 to JP16, JP14 to JP17, JP15 to JP18, JP16 to JP19, JP17 to JP20, JP18 to JP21, JP19 to JP22, JP20 to JP23, JP21 to JP24, JP22 to JP25, R18 to R20, R19 to R21, R20 to R22, R21 to R23, R22 to R24, R23 to R25
Connections:
- net 3V3_BUCK_VIN: now also C19.1, R19.2
- net 5V_BUCK_VIN: now also C14.1, C18.1, R18.2
- net GND: now also C14.2, C18.2, C19.2
- net at U7.5 (EN): now also R19.1
- net at U6.5 (EN): now also R18.1
