File: pcb/power_regulation.kicad_sch (KiCad schematic)
At the start: 46 parts, among them U6 TPS563201, U7 TPS563201, U8 LM1085-5.0, U9 LM1117IMPX-3.3

Commit message: Move audio jack (J6) into SA818V sheet, rename nets/jumpers for clarity
Relocates the switched TRS jack from audio.kicad_sch into SA818V.kicad_sch
and updates the root sheet's pin interface to match (SA818_IN_MIC,
SA818_IN_PTT, new SA818_IN_PTT_HB), fixing an I2C_MIC_OUT/I2S_MIC_OUT
naming typo along the way. Ring/ring-switch/sleeve are wired; tip and
tip-switch (mic audio leg) are still open, per audio_ptt_path.md.

Also: renames GPS hierarchical labels and several power/regulation/
peripheral jumper values from generic (Jumper_2_Open, SolderJumper_2_Open)
to descriptive names, wires MCU_OUT_PTT_HB, and removes now-unused test
points/jumpers from the battery input sheets. Adds 74hc123_pinout.md
planning doc for the TX-safety timeout / force-off failsafe part.

Co-Authored-By: Claude Sonnet 5 <noreply@anthropic.com>
Claude-Session: https://claude.ai/code/session_01P3G1ionr2QCR8SZtKRreL3
Parts:
- JP13: value SolderJumper_2_Open -> 5V ISO
- JP15: value SolderJumper_2_Open -> 3.3V ISO
- JP17: value SolderJumper_2_Open -> 5V LDO ISO
- JP19: value SolderJumper_2_Open -> 3.3V LDO ISO
- JP20: value Jumper_2_Open -> 5V TEST LOAD
- JP21: value Jumper_2_Open -> 3.3V TEST LOAD
- JP23: value SolderJumper_2_Open -> 5V LDO OUT
- JP25: value SolderJumper_2_Open -> 3.3V LDO OUT
Changed lines of the file:
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@@
 			)
 		)
-		(property "Value" "SolderJumper_2_Open"
+		(property "Value" "5V ISO"
 			(at 26.67 62.23 0)
 			(show_name no)
@@
 			)
 		)
-		(property "Value" "SolderJumper_2_Open"
+		(property "Value" "3.3V LDO ISO"
 			(at 177.8 134.62 0)
 			(show_name no)
@@
 			)
 		)
-		(property "Value" "Jumper_2_Open"
+		(property "Value" "3.3V TEST LOAD"
 			(at 252.73 146.0499 90)
 			(show_name no)
@@
 			)
 		)
-		(property "Value" "SolderJumper_2_Open"
+		(property "Value" "3.3V LDO OUT"
 			(at 261.62 134.62 0)
 			(show_name no)
@@
 		(property "Value" "Jumper_2_Open"
 			(at 177.8 125.73 0)
+			(hide yes)
 			(show_name no)
 			(do_not_autoplace no)
@@
 			)
 		)
-		(property "Value" "SolderJumper_2_Open"
+		(property "Value" "5V LDO OUT"
 			(at 257.81 57.15 0)
 			(show_name no)
@@
 		(property "Value" "Jumper_2_Open"
 			(at 27.94 130.81 0)
+			(hide yes)
 			(show_name no)
 			(do_not_autoplace no)
@@
 			)
 		)
-		(property "Value" "SolderJumper_2_Open"
+		(property "Value" "5V LDO ISO"
 			(at 176.53 57.15 0)
 			(show_name no)
@@
 			)
 		)
-		(property "Value" "SolderJumper_2_Open"
+		(property "Value" "3.3V ISO"
 			(at 27.94 139.7 0)
 			(show_name no)
@@
 		(property "Value" "Jumper_2_Open"
 			(at 176.53 46.99 0)
+			(hide yes)
 			(show_name no)
 			(do_not_autoplace no)
@@
 		(property "Value" "Jumper_2_Open"
 			(at 257.81 48.26 0)
+			(hide yes)
 			(show_name no)
 			(do_not_autoplace no)
@@
 			)
 		)
-		(property "Value" "Jumper_2_Open"
+		(property "Value" "5V TEST LOAD"
 			(at 248.92 71.1199 90)
 			(show_name no)
@@
 		(property "Value" "Jumper_2_Open"
 			(at 26.67 53.34 0)
+			(hide yes)
 			(show_name no)
 			(do_not_autoplace no)
