File: pcb/power_regulation.kicad_sch (KiCad schematic)
At the start: 46 parts, among them U6 TPS563201, U7 TPS563201, U8 LM1085-5.0, U9 LM1117IMPX-3.3

Commit message: annotations
Changed lines of the file:
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@@
 		(property "Value" "PWR_FLAG"
 			(at 195.58 55.88 0)
+			(hide yes)
 			(show_name no)
 			(do_not_autoplace no)
@@
 		(property "Value" "PWR_FLAG"
 			(at 66.04 138.43 0)
+			(hide yes)
 			(show_name no)
 			(do_not_autoplace no)
@@
 		(property "Value" "PWR_FLAG"
 			(at 64.77 60.96 0)
+			(hide yes)
 			(show_name no)
 			(do_not_autoplace no)
@@
 		(property "Value" "PWR_FLAG"
 			(at 198.12 133.35 0)
+			(hide yes)
 			(show_name no)
 			(do_not_autoplace no)

Commit message: changes on pcb
Parts:
- removed JP13: 5V ISO, Jumper:SolderJumper-2_P1.3mm_Open_TrianglePad1.0x1.5mm, symbol Jumper:SolderJumper_2_Open
- removed JP15: 3.3V ISO, Jumper:SolderJumper-2_P1.3mm_Open_TrianglePad1.0x1.5mm, symbol Jumper:SolderJumper_2_Open
- removed JP17: 5V LDO ISO, Jumper:SolderJumper-2_P1.3mm_Open_TrianglePad1.0x1.5mm, symbol Jumper:SolderJumper_2_Open
- removed JP19: 3.3V LDO ISO, Jumper:SolderJumper-2_P1.3mm_Open_TrianglePad1.0x1.5mm, symbol Jumper:SolderJumper_2_Open
- removed JP23: 5V LDO OUT, Jumper:SolderJumper-2_P1.3mm_Open_TrianglePad1.0x1.5mm, symbol Jumper:SolderJumper_2_Open
- removed JP25: 3.3V LDO OUT, Jumper:SolderJumper-2_P1.3mm_Open_TrianglePad1.0x1.5mm, symbol Jumper:SolderJumper_2_Open
- U9: footprint Package_TO_SOT_SMD:SOT-223 -> Package_TO_SOT_SMD:SOT-223-3_TabPin2
Connections:
- net 6V_intermediate: now reaches C20.1, L1.1, U6.2 (SW)
- net 4.8V_Intermediate: now reaches C21.1, L2.1, U7.2 (SW)
Other:
- note added: "4.78V Intermediate Power"
- moved on the sheet: JP12, JP14, JP16, JP18, JP22, JP24
