File: pcb/usbc-programming-uart.kicad_sch (KiCad schematic)
At the start: 14 parts, among them J6 HC-TYPE-C-16P-01A, Q5 MMBT2222A, Q6 MMBT2222A, SW1 RST, SW2 BOOT, U9 CH340C

Commit message: working through usb-c and hub
Parts:
- added C30, C31, C32, C34: 0.1u/25V, Capacitor_SMD:C_0603_1608Metric, symbol Device:C_Small
- added C33: 22u/16V Elec, Capacitor_SMD:C_Elec_5x5.8, symbol Device:C_Small
- added C36: 10u/25V, Capacitor_SMD:C_0805_2012Metric, symbol Device:C_Small
- added C37: 1u/25V, Capacitor_SMD:C_0805_2012Metric, symbol Device:C_Small
- added U10: AMS1117-3.3, Package_TO_SOT_SMD:SOT-223-3_TabPin2, symbol Regulator_Linear:AMS1117-3.3
- added U11: CH334R, Package_SO:QSOP-16_3.9x4.9mm_P0.635mm, symbol Interface_USB:CH334R
- added Y1: 12MHz, Crystal:Crystal_SMD_2520-4Pin_2.5x2.0mm, symbol PCM_SparkFun-Clock:Crystal
- J6: symbol Connector:USB_C_Receptacle_USB2.0_16P -> Connector:USB_C_Receptacle_USB2.0_14P
Connections:
- net GND: now also C30.1, C31.2, C32.2, C33.2, C34.2, C36.2, C37.2, U10.1 (GND), U11.14 (GND)
- net VBUS: now also U9.4 (V3), C30.2, C31.1, C37.1, U10.3 (VI), U11.12 (V5)
- net ~DTR: now reaches Q6.2 (E), R20.2, U9.13 (~{DTR})
- net ~RTS: now reaches Q5.2 (E), R21.2, U9.14 (~{RTS})
- net at J6.A6 (D+), J6.B6 (D+): now also U11.11 (DPU+); no longer U9.5 (UD+)
- net at J6.A7 (D-), J6.B7 (D-): now also U11.10 (DMU-); no longer U9.6 (UD-)
- new net: C34.1, C36.1, U11.13 (VDD33_{LDO})
- new net: U11.16 (XI), Y1.1
- new net: U11.15 (XO), Y1.2
- new net: U11.6 (DP2+), U9.5 (UD+)
- new net: U11.5 (DM2-), U9.6 (UD-)
- new net USB_3.3V: C32.1, C33.1, U10.2 (VO)
- new net USB_MCU_D+: U11.8 (DP1+)
- new net USB_MCU_D-: U11.7 (DM1-)
- no-connect marks 7 -> 10
Other:
- moved on the sheet: C27, C28, C29, Q5, Q6, R17, R18, R19, R20, R21, SW1, SW2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
