File: pcb/usbc-programming-uart.kicad_sch (KiCad schematic)
At the start: 27 parts, among them J3 HC-TYPE-C-16P-01A, Q3 MMBT2222A, Q4 MMBT2222A, SW1 RST, SW2 BOOT, U11 CH334R, U12 LM1117IMPX-3.3, U13 CH340C, Y1 12MHz

Commit message: Fix remaining mass-symbol-update reversions (67 Datasheet + 5 Footprint fields)
The project-wide "Update Symbols from Library" run reverted far more than
the 4 caught in the previous commit -- most of that commit's own claimed
"localized project-wide" state was actually already the reverted state,
since the mass update happened before that commit and git history alone
couldn't detect it. Cross-referenced every component's Datasheet/Footprint
against the independent tracking docs (project_library_datasheets.md,
kicad_gx_library_datasheets.md, footprint_verification_log.md) instead.

- 67 components: Datasheet reverted from a localized ${KIPRJMOD} path back
  to a remote URL, across all 8 schematic files
- 5 components: Footprint also reverted, not just Datasheet -- Y2 (RTC
  crystal) reverted to a physically different package size (5.0x3.2mm vs.
  the real 3.2x1.5mm part); U9/U12 (LM1117 LDOs), U10 (ESP32-S3 module),
  and Y1 (12MHz crystal) reverted to differently-sourced but plausible
  footprints from a vendored library instead of the verified stock ones

No MPN/Manf/LCSC Part#/Value regressions found (checked all 185
components). ERC clean, same 15 pre-existing errors as before.

Co-Authored-By: Claude Sonnet 5 <noreply@anthropic.com>
Claude-Session: https://claude.ai/code/session_01LhLkuH6sQ5GbUZ61bG7p2h
Parts:
- U12: footprint PCM_SparkFun-Semiconductor-Standard:SOT-223-3_TabPin2 -> Package_TO_SOT_SMD:SOT-223
- Y1: footprint PCM_SparkFun-Clock:Crystal_SMD_5.0x3.2mm -> Crystal:Crystal_SMD_2520-4Pin_2.5x2.0mm
Changed lines of the file:
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@@
 			)
 		)
-		(property "Datasheet" "https://www.lcsc.com/datasheet/C14677.pdf"
+		(property "Datasheet" "${KIPRJMOD}/project_library/datasheets/YAGEO/RC0603JR-075K1L.pdf"
 			(at 58.42 36.83 0)
 			(hide yes)
@@
 			)
 		)
-		(property "Datasheet" "https://www.lcsc.com/datasheet/C22435898.pdf"
+		(property "Datasheet" "${KIPRJMOD}/project_library/datasheets/LUTE/0805L050_16XR.pdf"
 			(at 55.88 24.13 0)
 			(hide yes)
@@
 			)
 		)
-		(property "Datasheet" "https://www.lcsc.com/datasheet/C14677.pdf"
+		(property "Datasheet" "${KIPRJMOD}/project_library/datasheets/YAGEO/RC0603JR-075K1L.pdf"
 			(at 58.42 44.45 0)
 			(hide yes)
@@
 			)
 		)
-		(property "Datasheet" "https://assets.nexperia.com/documents/data-sheet/MMBT2222A.pdf"
+		(property "Datasheet" "${KIPRJMOD}/project_library/datasheets/onsemi/MMBT2222ALT1G.pdf"
 			(at 119.38 162.56 0)
 			(hide yes)
@@
 			)
 		)
-		(property "Footprint" "PCM_SparkFun-Clock:Crystal_SMD_5.0x3.2mm"
+		(property "Footprint" "Crystal:Crystal_SMD_2520-4Pin_2.5x2.0mm"
 			(at 93.98 80.01 0)
 			(hide yes)
@@
 			)
 		)
-		(property "Datasheet" "https://www.lcsc.com/datasheet/C284154.pdf"
+		(property "Datasheet" "${KIPRJMOD}/project_library/datasheets/Yajingxin/TXM12M0004252DBCEO00T.pdf"
 			(at 93.98 77.47 0)
 			(hide yes)
@@
 			)
 		)
-		(property "Datasheet" "https://www.lcsc.com/datasheet/C84376.pdf"
+		(property "Datasheet" "${KIPRJMOD}/project_library/datasheets/YAGEO/RC0805FR-0710KL.pdf"
 			(at 134.62 162.56 0)
 			(hide yes)
@@
 			)
 		)
-		(property "Footprint" "PCM_SparkFun-Semiconductor-Standard:SOT-223-3_TabPin2"
+		(property "Footprint" "Package_TO_SOT_SMD:SOT-223"
 			(at 237.49 45.72 0)
 			(hide yes)
@@
 			)
 		)
-		(property "Datasheet" "http://www.ti.com/lit/ds/symlink/lm1117.pdf"
+		(property "Datasheet" "${KIPRJMOD}/project_library/datasheets/TI/LM1117IMPX-3.3_NOPB.pdf"
 			(at 237.49 40.64 0)
 			(hide yes)
@@
 			)
 		)
-		(property "Datasheet" "https://datasheet.lcsc.com/szlcsc/Jiangsu-Qin-Heng-CH340C_C84681.pdf"
+		(property "Datasheet" "${KIPRJMOD}/project_library/datasheets/WCH/CH340C.pdf"
 			(at 218.694 106.426 0)
 			(hide yes)
@@
 			)
 		)
-		(property "Datasheet" "${KIPRJMOD}/project_library/datasheets/Murata_Electronics/GRM21BZ71E106KE15L.pdf"
+		(property "Datasheet" "${KIPRJMOD}/project_library/datasheets/Murata_Electronics/GRM21BR71H105KA12L.pdf"
 			(at 135.89 38.1 0)
 			(hide yes)
@@
 			)
 		)
-		(property "Datasheet" "https://www.lcsc.com/datasheet/C77083.pdf"
+		(property "Datasheet" "${KIPRJMOD}/project_library/datasheets/Murata_Electronics/GRM21BR71H105KA12L.pdf"
 			(at 66.04 144.78 0)
 			(hide yes)
@@
 			)
 		)
-		(property "Datasheet" "https://www.lcsc.com/datasheet/C83916.pdf"
+		(property "Datasheet" "${KIPRJMOD}/project_library/datasheets/Korean_Hroparts_Elec/K2-1102SP-A4SC-04.pdf"
 			(at 114.3 175.26 0)
 			(hide yes)
@@
 			)
 		)
-		(property "Datasheet" "https://www.lcsc.com/datasheet/C84376.pdf"
+		(property "Datasheet" "${KIPRJMOD}/project_library/datasheets/YAGEO/RC0805FR-0710KL.pdf"
 			(at 133.35 137.16 0)
 			(hide yes)
@@
 			)
 		)
-		(property "Datasheet" "https://www.lcsc.com/datasheet/C84376.pdf"
+		(property "Datasheet" "${KIPRJMOD}/project_library/datasheets/YAGEO/RC0805FR-0710KL.pdf"
 			(at 66.04 134.62 0)
 			(hide yes)
@@
 			)
 		)
-		(property "Datasheet" "https://www.wch-ic.com/download/file?id=327"
+		(property "Datasheet" "${KIPRJMOD}/project_library/datasheets/WCH/CH334R.pdf"
 			(at 119.38 29.21 0)
 			(hide yes)
@@
 			)
 		)
-		(property "Datasheet" "https://assets.nexperia.com/documents/data-sheet/MMBT2222A.pdf"
+		(property "Datasheet" "${KIPRJMOD}/project_library/datasheets/onsemi/MMBT2222ALT1G.pdf"
 			(at 119.38 137.16 0)
 			(hide yes)
@@
 			)
 		)
-		(property "Datasheet" "https://www.lcsc.com/datasheet/C83916.pdf"
+		(property "Datasheet" "${KIPRJMOD}/project_library/datasheets/Korean_Hroparts_Elec/K2-1102SP-A4SC-04.pdf"
 			(at 52.07 135.89 0)
 			(hide yes)
