File: pcb/usbc-programming-uart.kicad_sch (KiCad schematic)
At the start: 27 parts, among them J3 HC-TYPE-C-16P-01A, Q3 MMBT2222A, Q4 MMBT2222A, SW1 RST, SW2 BOOT, U11 CH334R, U12 LM1117IMPX-3.3, U13 CH340C, Y1 12MHz

Commit message: change some 0805s to 0603
Parts:
- removed R26, R27, R28: 10k, Resistor_SMD:R_0805_2012Metric, symbol Device:R_US
- added R32, R33, R34: 10k, Resistor_SMD:R_0603_1608Metric, symbol Device:R_US
- renumbered C31 to C35, C32 to C36, C33 to C37, C34 to C38, C35 to C39, C36 to C40, C38 to C41, C41 to C42, C37 to C43, C39 to C44, C40 to C45, J3 to J4, JP24 to JP26, Q3 to Q6, Q4 to Q7, R24 to R30, R25 to R31, SW1 to SW2, SW2 to SW3, U13 to U12, U12 to U13
Connections:
- net +3.3V: now also R32.2
- net MCU_EN_RESET: now also R32.1
- net ~DTR: now also R33.1
- net ~RTS: now also R34.1
- net at Q7.1 (B): now also R34.2
- net at Q6.1 (B): now also R33.2
