File: pcb/usbc-programming-uart.kicad_sch (KiCad schematic)
At the start: 27 parts, among them J4 HC-TYPE-C-16P-01A, Q6 MMBT2222A, Q7 MMBT2222A, SW2 RST, SW3 BOOT, U11 CH334R, U12 CH340C, U13 LM1117IMPX-3.3, Y1 12MHz

Commit message: Move audio jack (J6) into SA818V sheet, rename nets/jumpers for clarity
Relocates the switched TRS jack from audio.kicad_sch into SA818V.kicad_sch
and updates the root sheet's pin interface to match (SA818_IN_MIC,
SA818_IN_PTT, new SA818_IN_PTT_HB), fixing an I2C_MIC_OUT/I2S_MIC_OUT
naming typo along the way. Ring/ring-switch/sleeve are wired; tip and
tip-switch (mic audio leg) are still open, per audio_ptt_path.md.

Also: renames GPS hierarchical labels and several power/regulation/
peripheral jumper values from generic (Jumper_2_Open, SolderJumper_2_Open)
to descriptive names, wires MCU_OUT_PTT_HB, and removes now-unused test
points/jumpers from the battery input sheets. Adds 74hc123_pinout.md
planning doc for the TX-safety timeout / force-off failsafe part.

Co-Authored-By: Claude Sonnet 5 <noreply@anthropic.com>
Claude-Session: https://claude.ai/code/session_01P3G1ionr2QCR8SZtKRreL3
Parts:
- JP26: value Jumper_2_Open -> USB Power Enable
Changed lines of the file:
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@@
 			)
 		)
-		(property "Value" "Jumper_2_Open"
+		(property "Value" "USB Power Enable"
 			(at 179.07 19.05 0)
 			(show_name no)
