File: pcb/battery_18650_input.kicad_sch (KiCad schematic)
At the start: 21 parts, among them Q1 AO3400A, Q2 8205A, U5 MAX17320

Commit message: updated battery regulation circuit to bump up intermediate voltages
Parts:
- R13: footprint Resistor_SMD:R_Shunt_Vishay_WSK2512_6332Metric_T2.21mm -> kicad_gx_library:RES-SMD_L6.4-W3.2-R2512_Sense4Pin
Changed lines of the file:
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@@
 			)
 		)
-		(property "Footprint" "Resistor_SMD:R_Shunt_Vishay_WSK2512_6332Metric_T2.21mm"
+		(property "Footprint" "kicad_gx_library:RES-SMD_L6.4-W3.2-R2512_Sense4Pin"
 			(at 152.4 130.048 90)
 			(hide yes)
