File: pcb/battery_18650_input.kicad_sch (KiCad schematic)
At the start: 21 parts, among them Q1 AO3400A, Q2 8205A, U5 MAX17320

Commit message: change some 0805s to 0603
Parts:
- renumbered C8 to C10, C9 to C11, C4 to C6, C5 to C7, C6 to C8, C7 to C9, Q1 to Q2, Q2 to Q3, R10 to R12, R11 to R13, R12 to R14, R13 to R15, R14 to R16, R15 to R17
