File: pcb/battery_18650_input.kicad_sch (KiCad schematic)
At the start: 19 parts, among them Q2 AO3400A, Q3 8205A, U5 MAX17320

Commit message: annotations
Other:
- note added: "18650s"
- moved on the sheet: BT2, R14
Changed lines of the file:
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@@
 	(generator_version "10.0")
 	(paper "A4")
+	(rectangle
+		(start 58.42 85.09)
+		(end 90.17 111.76)
+		(stroke
+			(width 0)
+			(type default)
+		)
+		(fill
+			(type none)
+		)
+	)
+	(text "18650s"
+		(exclude_from_sim no)
+		(at 64.516 87.122 0)
+		(effects
+			(font
+				(size 1.27 1.27)
+			)
+		)
+	)
 	(text "R13: intentional GND/GNDREF split for current sensing — do not bridge elsewhere"
 		(exclude_from_sim no)
@@
 	)
 	(junction
-		(at 72.39 86.36)
+		(at 72.39 63.5)
 		(diameter 0)
 		(color 0 0 0 0)
@@
 	(wire
 		(pts
-			(xy 72.39 72.39) (xy 72.39 80.01)
+			(xy 72.39 59.69) (xy 72.39 87.63)
 		)
 		(stroke
@@
 	(wire
 		(pts
-			(xy 66.04 85.09) (xy 66.04 86.36)
-		)
-		(stroke
-			(width 0)
-			(type default)
-		)
-	)
-	(wire
-		(pts
 			(xy 154.94 121.92) (xy 154.94 125.73)
 		)
@@
 	(wire
 		(pts
-			(xy 72.39 97.79) (xy 86.36 97.79)
+			(xy 72.39 97.79) (xy 90.17 97.79)
 		)
 		(stroke
@@
 	(wire
 		(pts
-			(xy 93.98 97.79) (xy 102.87 97.79)
+			(xy 97.79 97.79) (xy 102.87 97.79)
 		)
 		(stroke
@@
 	(wire
 		(pts
-			(xy 66.04 86.36) (xy 72.39 86.36)
+			(xy 71.12 63.5) (xy 72.39 63.5)
 		)
 		(stroke
@@
 	(wire
 		(pts
-			(xy 72.39 107.95) (xy 72.39 128.27)
+			(xy 72.39 109.22) (xy 72.39 128.27)
 		)
 		(stroke
@@
 	(wire
 		(pts
-			(xy 72.39 80.01) (xy 72.39 86.36)
-		)
-		(stroke
-			(width 0)
-			(type default)
-		)
-	)
-	(wire
-		(pts
 			(xy 107.95 72.39) (xy 107.95 81.28)
 		)
@@
 	(wire
 		(pts
-			(xy 72.39 86.36) (xy 72.39 87.63)
-		)
-		(stroke
-			(width 0)
-			(type default)
-		)
-	)
-	(wire
-		(pts
 			(xy 149.86 62.23) (xy 149.86 64.77)
 		)
@@
 	(wire
 		(pts
-			(xy 72.39 59.69) (xy 72.39 72.39)
-		)
-		(stroke
-			(width 0)
-			(type default)
-		)
-	)
-	(wire
-		(pts
 			(xy 113.03 87.63) (xy 113.03 88.9)
 		)
@@
 	(wire
 		(pts
-			(xy 72.39 97.79) (xy 72.39 100.33)
+			(xy 72.39 97.79) (xy 72.39 101.6)
 		)
 		(stroke
@@
 		(property "Value" "PWR_FLAG"
 			(at 194.31 41.91 0)
+			(hide yes)
 			(show_name no)
 			(do_not_autoplace no)
@@
 		(property "Value" "PWR_FLAG"
 			(at 116.332 67.31 90)
+			(hide yes)
 			(show_name no)
 			(do_not_autoplace no)
@@
 	(symbol
 		(lib_id "Device:Battery_Cell")
-		(at 72.39 105.41 0)
+		(at 72.39 106.68 0)
 		(unit 1)
 		(body_style 1)
@@
 		(fields_autoplaced yes)
 		(property "Reference" "BT2"
-			(at 76.2 102.2984 0)
+			(at 76.2 103.5684 0)
 			(show_name no)
 			(do_not_autoplace no)
@@
 		)
 		(property "Value" "Battery_Cell"
-			(at 76.2 104.8384 0)
+			(at 76.2 106.1084 0)
 			(show_name no)
 			(do_not_autoplace no)
@@
 		)
 		(property "Footprint" "Battery:BatteryHolder_MPD_BH-18650-PC"
-			(at 72.39 103.886 90)
+			(at 72.39 105.156 90)
 			(hide yes)
 			(show_name no)
@@
 		)
 		(property "Datasheet" "${KIPRJMOD}/project_library/datasheets/MPD/BH-18650-PC.pdf"
-			(at 72.39 103.886 90)
+			(at 72.39 105.156 90)
 			(hide yes)
 			(show_name no)
@@
 		)
 		(property "Description" "Single-cell battery"
-			(at 72.39 105.41 0)
+			(at 72.39 106.68 0)
 			(hide yes)
 			(show_name no)
@@
 		)
 		(property "Sim.Device" "V"
-			(at 72.39 105.41 0)
+			(at 72.39 106.68 0)
 			(hide yes)
 			(show_name no)
@@
 		)
 		(property "Sim.Type" "DC"
-			(at 72.39 105.41 0)
+			(at 72.39 106.68 0)
 			(hide yes)
 			(show_name no)
@@
 		)
 		(property "Sim.Pins" "1=+ 2=-"
-			(at 72.39 105.41 0)
+			(at 72.39 106.68 0)
 			(hide yes)
 			(show_name no)
@@
 		)
 		(property "LCSC Part #" "C5339083"
-			(at 72.39 105.41 0)
+			(at 72.39 106.68 0)
 			(hide yes)
 			(show_name no)
@@
 		)
 		(property "Manf" "MPD (Memory Protection Devices)"
-			(at 72.39 105.41 0)
+			(at 72.39 106.68 0)
 			(hide yes)
 			(show_name no)
@@
 		)
 		(property "MPN" "BH-18650-PC"
-			(at 72.39 105.41 0)
+			(at 72.39 106.68 0)
 			(hide yes)
 			(show_name no)
@@
 		)
 		(property "Field10" ""
-			(at 72.39 105.41 0)
+			(at 72.39 106.68 0)
 			(hide yes)
 			(show_name no)
@@
 		(property "Value" "PWR_FLAG"
 			(at 133.35 41.91 0)
+			(hide yes)
 			(show_name no)
 			(do_not_autoplace no)
@@
 	(symbol
 		(lib_id "Device:R_US")
-		(at 90.17 97.79 90)
+		(at 93.98 97.79 90)
 		(unit 1)
 		(body_style 1)
@@
 		(dnp no)
 		(property "Reference" "R14"
-			(at 89.916 96.012 90)
+			(at 93.726 96.012 90)
 			(show_name no)
 			(do_not_autoplace no)
@@
 		)
 		(property "Value" "150"
-			(at 90.424 99.822 90)
+			(at 94.234 99.822 90)
 			(show_name no)
 			(do_not_autoplace no)
@@
 		)
 		(property "Footprint" "Resistor_SMD:R_1206_3216Metric"
-			(at 90.424 96.774 90)
+			(at 94.234 96.774 90)
 			(hide yes)
 			(show_name no)
@@
 		)
 		(property "Datasheet" "${KIPRJMOD}/project_library/datasheets/YAGEO/RT1206BRD07150RL.pdf"
-			(at 90.17 97.79 0)
+			(at 93.98 97.79 0)
 			(hide yes)
 			(show_name no)
@@
 		)
 		(property "Description" "Resistor, US symbol"
-			(at 90.17 97.79 0)
+			(at 93.98 97.79 0)
 			(hide yes)
 			(show_name no)
@@
 		)
 		(property "PROD_ID" "RES-07856"
-			(at 97.028 97.79 0)
+			(at 100.838 97.79 0)
 			(hide yes)
 			(show_name no)
@@
 		)
 		(property "LCSC Part #" "C870430"
-			(at 90.17 97.79 0)
+			(at 93.98 97.79 0)
 			(hide yes)
 			(show_name no)
@@
 		)
 		(property "Manf" "YAGEO"
-			(at 90.17 97.79 0)
+			(at 93.98 97.79 0)
 			(hide yes)
 			(show_name no)
@@
 		)
 		(property "MPN" "RT1206BRD07150RL"
-			(at 90.17 97.79 0)
+			(at 93.98 97.79 0)
 			(hide yes)
 			(show_name no)
@@
 		)
 		(property "Field10" ""
-			(at 90.17 97.79 90)
+			(at 93.98 97.79 90)
 			(hide yes)
 			(show_name no)
@@
 		(property "Value" "PWR_FLAG"
 			(at 187.96 123.19 0)
+			(hide yes)
 			(show_name no)
 			(do_not_autoplace no)
@@
 	(symbol
 		(lib_id "power:PWR_FLAG")
-		(at 66.04 85.09 0)
+		(at 71.12 63.5 90)
 		(unit 1)
 		(body_style 1)
@@
 		(fields_autoplaced yes)
 		(property "Reference" "#FLG07"
-			(at 66.04 83.185 0)
+			(at 69.215 63.5 0)
 			(hide yes)
 			(show_name no)
@@
 		)
 		(property "Value" "PWR_FLAG"
-			(at 66.04 80.01 0)
+			(at 66.04 63.5 0)
+			(hide yes)
 			(show_name no)
 			(do_not_autoplace no)
@@
 		)
 		(property "Footprint" ""
-			(at 66.04 85.09 0)
+			(at 71.12 63.5 0)
 			(hide yes)
 			(show_name no)
@@
 		)
 		(property "Datasheet" ""
-			(at 66.04 85.09 0)
+			(at 71.12 63.5 0)
 			(hide yes)
 			(show_name no)
@@
 		)
 		(property "Description" "Special symbol for telling ERC where power comes from"
-			(at 66.04 85.09 0)
+			(at 71.12 63.5 0)
 			(hide yes)
 			(show_name no)

Commit message: changes on pcb
Parts:
- BT1, BT2: footprint Battery:BatteryHolder_MPD_BH-18650-PC -> kicad_gx_library:BatteryHolder_MPD_BH-18650-PC
Connections:
- net PolyFuseOut: now reaches F1.3, Q3.1 (S1)
- net BATT_Plus_to_Minus: now reaches BT1.2 (-), BT2.1 (+), R14.1
- net +BATT renamed BATT+
Changed lines of the file:
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@@
-	)
-	(junction
-		(at 72.39 59.69)
-		(diameter 0)
-		(color 0 0 0 0)
 	)
 	(junction
@@
 	(wire
 		(pts
-			(xy 72.39 59.69) (xy 72.39 87.63)
+			(xy 72.39 46.99) (xy 72.39 87.63)
 		)
 		(stroke
@@
 	(wire
 		(pts
-			(xy 110.49 46.99) (xy 87.63 46.99)
-		)
-		(stroke
-			(width 0)
-			(type default)
-		)
-	)
-	(wire
-		(pts
 			(xy 187.96 128.27) (xy 187.96 130.81)
 		)
@@
 	(wire
 		(pts
-			(xy 72.39 55.88) (xy 72.39 59.69)
-		)
-		(stroke
-			(width 0)
-			(type default)
-		)
-	)
-	(wire
-		(pts
 			(xy 142.24 62.23) (xy 142.24 68.58)
 		)
@@
 	(wire
 		(pts
-			(xy 87.63 46.99) (xy 87.63 59.69)
-		)
-		(stroke
-			(width 0)
-			(type default)
-		)
-	)
-	(wire
-		(pts
 			(xy 130.81 90.17) (xy 121.92 90.17)
 		)
@@
 	(wire
 		(pts
-			(xy 87.63 59.69) (xy 72.39 59.69)
+			(xy 72.39 46.99) (xy 110.49 46.99)
 		)
 		(stroke
@@
 			(width 0)
 			(type default)
+		)
+	)
+	(label "BATT_Plus_to_Minus"
+		(at 73.66 97.79 0)
+		(effects
+			(font
+				(size 1.27 1.27)
+			)
+			(justify left bottom)
+		)
+	)
+	(label "PolyFuseOut"
+		(at 120.65 46.99 0)
+		(effects
+			(font
+				(size 1.27 1.27)
+			)
+			(justify left bottom)
+		)
+	)
+	(label "BATT+"
+		(at 80.01 46.99 0)
+		(effects
+			(font
+				(size 1.27 1.27)
+			)
+			(justify left bottom)
 		)
 	)
@@
 			)
 		)
-		(property "Footprint" "Battery:BatteryHolder_MPD_BH-18650-PC"
+		(property "Footprint" "kicad_gx_library:BatteryHolder_MPD_BH-18650-PC"
 			(at 72.39 91.186 90)
 			(hide yes)
@@
 	)
 	(symbol
-		(lib_id "power:+BATT")
-		(at 72.39 55.88 0)
-		(unit 1)
-		(body_style 1)
-		(exclude_from_sim no)
-		(in_bom yes)
-		(on_board yes)
-		(in_pos_files yes)
-		(dnp no)
-		(fields_autoplaced yes)
-		(property "Reference" "#PWR030"
-			(at 72.39 59.69 0)
-			(hide yes)
-			(show_name no)
-			(do_not_autoplace no)
-			(effects
-				(font
-					(size 1.27 1.27)
-				)
-			)
-		)
-		(property "Value" "+BATT"
-			(at 72.39 50.8 0)
-			(show_name no)
-			(do_not_autoplace no)
-			(effects
-				(font
-					(size 1.27 1.27)
-				)
-			)
-		)
-		(property "Footprint" ""
-			(at 72.39 55.88 0)
-			(hide yes)
-			(show_name no)
-			(do_not_autoplace no)
-			(effects
-				(font
-					(size 1.27 1.27)
-				)
-			)
-		)
-		(property "Datasheet" ""
-			(at 72.39 55.88 0)
-			(hide yes)
-			(show_name no)
-			(do_not_autoplace no)
-			(effects
-				(font
-					(size 1.27 1.27)
-				)
-			)
-		)
-		(property "Description" "Power symbol creates a global label with name \"+BATT\""
-			(at 72.39 55.88 0)
-			(hide yes)
-			(show_name no)
-			(do_not_autoplace no)
-			(effects
-				(font
-					(size 1.27 1.27)
-				)
-			)
-		)
-		(pin "1"
-		)
-		(instances
-			(project "foxhunt1"
-				(path "/8399ba4b-9428-480d-8b65-76cf154b97a5/37ac1273-0b70-4a42-ac28-8e382584c4a4/c9765cc1-b0b1-40a4-af82-69bea9af9891"
-					(reference "#PWR030")
-					(unit 1)
-				)
-			)
-		)
-	)
-	(symbol
 		(lib_id "Device:Thermistor_US")
 		(at 118.11 116.84 0)
@@
 			)
 		)
-		(property "Footprint" "Battery:BatteryHolder_MPD_BH-18650-PC"
+		(property "Footprint" "kicad_gx_library:BatteryHolder_MPD_BH-18650-PC"
 			(at 72.39 105.156 90)
 			(hide yes)
