File: pcb/peripherals.kicad_sch (KiCad schematic)
At the start: 39 parts, among them J4 Conn_01x03, J5 Conn_01x03, J6 Conn_01x03, J7 Conn_01x03, Q7 BSS138, Q8 AO3407A, SW10 GENERAL, SW4 SW_DIP_x04, SW7 GENERAL, SW8 GENERAL, SW9 GENERAL, U14 PCF8563T, U15 PCA9555PW, Y2 32.768kHz 9pF

Commit message: fix some drc issues
Parts:
- D2, D3: footprint Package_TO_SOT_SMD:TSOT-23 -> kicad_gx_library:SOT-23_L2.9-W1.3-P1.90-LS2.4-BR; Imported (none) -> 2026-09-19; LCSC Part (none) -> C232527; Manufacturer (none) -> onsemi; Modified (none) -> 2026-09-20; Source (none) -> easyeda2kicad
Changed lines of the file:
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@@
 			)
 		)
-		(property "Footprint" "Package_TO_SOT_SMD:TSOT-23"
+		(property "Footprint" "kicad_gx_library:SOT-23_L2.9-W1.3-P1.90-LS2.4-BR"
 			(at 66.04 31.115 0)
 			(hide yes)
@@
 			)
 		)
-		(property "Datasheet" "https://www.lcsc.com/datasheet/C232527.pdf"
+		(property "Datasheet" "https://lcsc.com/product-detail/Switching-Diode_ON-Semicon_BAS116LT1G_ON-Semicon-ON-BAS116LT1G_C232527.html"
 			(at 66.04 35.56 0)
 			(hide yes)
@@
 		)
 		(property "Package" "SOT-23"
+			(at 66.04 35.56 0)
+			(hide yes)
+			(show_name no)
+			(do_not_autoplace no)
+			(effects
+				(font
+					(size 1.27 1.27)
+				)
+			)
+		)
+		(property "Manufacturer" "onsemi"
+			(at 66.04 20.32 0)
+			(hide yes)
+			(show_name no)
+			(do_not_autoplace no)
+			(effects
+				(font
+					(size 1.27 1.27)
+				)
+			)
+		)
+		(property "LCSC Part" "C232527"
+			(at 66.04 15.24 0)
+			(hide yes)
+			(show_name no)
+			(do_not_autoplace no)
+			(effects
+				(font
+					(size 1.27 1.27)
+				)
+			)
+		)
+		(property "Source" "easyeda2kicad"
+			(at 66.04 10.16 0)
+			(hide yes)
+			(show_name no)
+			(do_not_autoplace no)
+			(effects
+				(font
+					(size 1.27 1.27)
+				)
+			)
+		)
+		(property "Imported" "2026-09-19"
+			(at 66.04 7.62 0)
+			(hide yes)
+			(show_name no)
+			(do_not_autoplace no)
+			(effects
+				(font
+					(size 1.27 1.27)
+				)
+			)
+		)
+		(property "Modified" "2026-09-20"
 			(at 66.04 35.56 0)
 			(hide yes)
@@
 			)
 		)
-		(property "Footprint" "Package_TO_SOT_SMD:TSOT-23"
+		(property "Footprint" "kicad_gx_library:SOT-23_L2.9-W1.3-P1.90-LS2.4-BR"
 			(at 50.8 45.085 0)
 			(hide yes)
@@
 			)
 		)
-		(property "Datasheet" "https://www.lcsc.com/datasheet/C232527.pdf"
+		(property "Datasheet" "https://lcsc.com/product-detail/Switching-Diode_ON-Semicon_BAS116LT1G_ON-Semicon-ON-BAS116LT1G_C232527.html"
 			(at 50.8 40.64 0)
 			(hide yes)
@@
 			(at 50.8 40.64 0)
 			(hide yes)
+			(show_name no)
+			(do_not_autoplace no)
+			(effects
+				(font
+					(size 1.27 1.27)
+				)
+			)
+		)
+		(property "Manufacturer" "onsemi"
+			(at 50.8 55.88 0)
+			(hide yes)
+			(show_name no)
+			(do_not_autoplace no)
+			(effects
+				(font
+					(size 1.27 1.27)
+				)
+			)
+		)
+		(property "LCSC Part" "C232527"
+			(at 50.8 60.96 0)
+			(hide yes)
+			(show_name no)
+			(do_not_autoplace no)
+			(effects
+				(font
+					(size 1.27 1.27)
+				)
+			)
+		)
+		(property "Source" "easyeda2kicad"
+			(at 50.8 66.04 0)
+			(hide yes)
+			(show_name no)
+			(do_not_autoplace no)
+			(effects
+				(font
+					(size 1.27 1.27)
+				)
+			)
+		)
+		(property "Imported" "2026-09-19"
+			(at 50.8 68.58 0)
+			(hide yes)
+			(show_name no)
+			(do_not_autoplace no)
+			(effects
+				(font
+					(size 1.27 1.27)
+				)
+			)
+		)
+		(property "Modified" "2026-09-20"
+			(at 50.8 40.64 0)
+			(hide yes)
