File: pcb/peripherals.kicad_sch (KiCad schematic)
At the start: 34 parts, among them Q7 BSS138, Q8 AO3407A, SW10 GENERAL, SW4 SW_DIP_x04, SW7 GENERAL, SW8 GENERAL, SW9 GENERAL, U14 PCF8563T, U15 PCA9555PW, U16 CAT24C32YI-GT3, Y2 32.768kHz 9pF

Commit message: change some 0805s to 0603
Parts:
- renumbered C43 to C46, C44 to C47, C51 to C48, C45 to C49, C46 to C50, C48 to C51, C47 to C52, C49 to C53, D2 to D4, D3 to D5, D10 to D6, D9 to D7, D7 to D9, Q7 to Q9, R30 to R35, R31 to R36, R35 to R37, R36 to R38, R37 to R39, R38 to R40, R34 to R41, SW7 to SW4, SW8 to SW5, SW10 to SW6, SW9 to SW7, SW4 to SW8, U16 to U14, U14 to U15, U15 to U16
