File: pcb/peripherals.kicad_sch (KiCad schematic)
At the start: 34 parts, among them Q8 AO3407A, Q9 BSS138, SW4 GENERAL, SW5 GENERAL, SW6 GENERAL, SW7 GENERAL, SW8 SW_DIP_x04, U14 CAT24C32YI-GT3, U15 PCF8563T, U16 PCA9555PW, Y2 32.768kHz 9pF

Commit message: Move audio jack (J6) into SA818V sheet, rename nets/jumpers for clarity
Relocates the switched TRS jack from audio.kicad_sch into SA818V.kicad_sch
and updates the root sheet's pin interface to match (SA818_IN_MIC,
SA818_IN_PTT, new SA818_IN_PTT_HB), fixing an I2C_MIC_OUT/I2S_MIC_OUT
naming typo along the way. Ring/ring-switch/sleeve are wired; tip and
tip-switch (mic audio leg) are still open, per audio_ptt_path.md.

Also: renames GPS hierarchical labels and several power/regulation/
peripheral jumper values from generic (Jumper_2_Open, SolderJumper_2_Open)
to descriptive names, wires MCU_OUT_PTT_HB, and removes now-unused test
points/jumpers from the battery input sheets. Adds 74hc123_pinout.md
planning doc for the TX-safety timeout / force-off failsafe part.

Co-Authored-By: Claude Sonnet 5 <noreply@anthropic.com>
Claude-Session: https://claude.ai/code/session_01P3G1ionr2QCR8SZtKRreL3
Parts:
- JP27: value SolderJumper_2_Open -> Write Protect
Changed lines of the file:
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@@
 			)
 		)
-		(property "Value" "SolderJumper_2_Open"
+		(property "Value" "Write Protect"
 			(at 83.82 163.068 0)
 			(show_name no)
