File: pcb/audio.kicad_sch (KiCad schematic)
At the start: 24 parts, among them J11 SJ2-3593D-SMT-TR, J9 Conn_01x03, U17 PCM5102A, U20 PC817C-S

Commit message: change some 0805s to 0603
Parts:
- renumbered C56 to C54, C54 to C56, C60 to C58, C63 to C59, C64 to C60, C58 to C61, C61 to C62, C59 to C63, C65 to C64, C62 to C65, J9 to J5, J11 to J6, R46 to R42, R47 to R43, R48 to R44, R49 to R45, R50 to R46, R55 to R47, R53 to R48, U20 to U18
