File: pcb/audio.kicad_sch (KiCad schematic)
At the start: 20 parts, among them J5 Conn_01x03, U17 PCM5102A

Commit message: annotations
Other:
- note added: "I2S AUDIO"
Changed lines of the file:
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@@
+		)
+	)
+	(text "I2S AUDIO"
+		(exclude_from_sim no)
+		(at 29.464 17.272 0)
+		(effects
+			(font
+				(size 3.81 3.81)
+			)
 		)
 	)
