File: pcb/gps.kicad_sch (KiCad schematic)
At the start: 18 parts, among them J10 RF_SMA, Q10 AO3407A, Q13 BSS138, U18 MAX-M10S

Commit message: change some 0805s to 0603
Parts:
- renumbered C68 to C67, C67 to C68, D6 to D10, D12 to D11, D11 to D12, J10 to J7, Q13 to Q10, Q10 to Q11, R56 to R49, R57 to R50, R41 to R51, R51 to R52, R52 to R53, U18 to U19
