File: pcb/gps.kicad_sch (KiCad schematic)
At the start: 18 parts, among them J7 RF_SMA, Q10 BSS138, Q11 AO3407A, U19 MAX-M10S

Commit message: Move audio jack (J6) into SA818V sheet, rename nets/jumpers for clarity
Relocates the switched TRS jack from audio.kicad_sch into SA818V.kicad_sch
and updates the root sheet's pin interface to match (SA818_IN_MIC,
SA818_IN_PTT, new SA818_IN_PTT_HB), fixing an I2C_MIC_OUT/I2S_MIC_OUT
naming typo along the way. Ring/ring-switch/sleeve are wired; tip and
tip-switch (mic audio leg) are still open, per audio_ptt_path.md.

Also: renames GPS hierarchical labels and several power/regulation/
peripheral jumper values from generic (Jumper_2_Open, SolderJumper_2_Open)
to descriptive names, wires MCU_OUT_PTT_HB, and removes now-unused test
points/jumpers from the battery input sheets. Adds 74hc123_pinout.md
planning doc for the TX-safety timeout / force-off failsafe part.

Co-Authored-By: Claude Sonnet 5 <noreply@anthropic.com>
Claude-Session: https://claude.ai/code/session_01P3G1ionr2QCR8SZtKRreL3
Parts:
- JP28: value Jumper_2_Open -> Bypass PWR SW
Connections:
- net PERIPH_OUT_GPS_EXTINT renamed GPS_IN_EXTINT
- net PERIPH_OUT_GPS_PWRON renamed GPS_IN_PWRON
Changed lines of the file:
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@@
 		)
 	)
-	(hierarchical_label "PERIPH_OUT_GPS_PWRON"
+	(hierarchical_label "GPS_IN_PWRON"
 		(shape input)
 		(at 78.74 57.15 180)
@@
 		)
 	)
-	(hierarchical_label "PERIPH_OUT_GPS_EXTINT"
+	(hierarchical_label "GPS_IN_EXTINT"
 		(shape input)
 		(at 93.98 93.98 180)
@@
 			)
 		)
-		(property "Value" "Jumper_2_Open"
-			(at 134.62 35.814 0)
-			(show_name no)
-			(do_not_autoplace no)
+		(property "Value" "Bypass PWR SW"
+			(at 135.636 36.068 0)
+			(show_name no)
+			(do_not_autoplace no)
