File: pcb/gps.kicad_sch (KiCad schematic)
At the start: 18 parts, among them J7 RF_SMA, Q10 BSS138, Q11 AO3407A, U19 MAX-M10S

Commit message: annotations
Other:
- note added: "GPS"
Changed lines of the file:
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@@
 	(generator_version "10.0")
 	(paper "A4")
+	(text "GPS"
+		(exclude_from_sim no)
+		(at 28.956 17.526 0)
+		(effects
+			(font
+				(size 3.81 3.81)
+			)
+		)
+	)
 	(junction
 		(at 181.61 88.9)

Commit message: module routing
Parts:
- J7: footprint Connector_Coaxial:SMA_Amphenol_132289_EdgeMount -> Connector_Coaxial:SMA_Amphenol_132134-11_Vertical
Changed lines of the file:
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@@
 			)
 		)
-		(property "Footprint" "Connector_Coaxial:SMA_Amphenol_132289_EdgeMount"
+		(property "Footprint" "Connector_Coaxial:SMA_Amphenol_132134-11_Vertical"
 			(at 200.66 88.9 0)
 			(hide yes)
