File: pcb/SA818V.kicad_sch (KiCad schematic)
At the start: 45 parts, among them J8 RF_SMA, J9 AudioJack, Q12 BSS138, Q13 BSS138, Q14 BSS138, U20 SA818S-V, U21 74HC123, U23 74LVC1G38, U24 74LVC1G38

Commit message: module routing
Parts:
- J8: footprint Connector_Coaxial:SMA_Amphenol_132289_EdgeMount -> Connector_Coaxial:SMA_Amphenol_132134-11_Vertical
Changed lines of the file:
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@@
 			)
 		)
-		(property "Footprint" "Connector_Coaxial:SMA_Amphenol_132289_EdgeMount"
+		(property "Footprint" "Connector_Coaxial:SMA_Amphenol_132134-11_Vertical"
 			(at 85.09 53.34 0)
 			(hide yes)
