File: pcb/foxhunt1.kicad_pcb (KiCad board)
At the start: 4 copper layers, 0 parts

Commit message: changes on pcb
Parts:
- added BT1: Battery_Cell, kicad_gx_library:BatteryHolder_MPD_BH-18650-PC, B.Cu at (62.4, 49.6)
- added BT2: Battery_Cell, kicad_gx_library:BatteryHolder_MPD_BH-18650-PC, B.Cu at (85.8, 49.6)
- added BT3: CR2032, kicad_gx_library:BAT-SMD_BS-08-B2AA016, B.Cu at (108.2, 116.1)
- added BT4: CR2032, kicad_gx_library:BAT-SMD_BS-08-B2AA016, B.Cu at (134.7, 72.8)
- added C1: 0.01u/25V, Capacitor_SMD:C_0603_1608Metric, F.Cu at (105.7, 92.5)
- added C10: 0.47u/10V, Capacitor_SMD:C_0603_1608Metric, F.Cu at (47.4, 68.4)
- added C11: 0.47u/10V, Capacitor_SMD:C_0603_1608Metric, F.Cu at (40.0, 65.8)
- added C12: 22u/16V, Capacitor_SMD:C_1206_3216Metric, F.Cu at (52.7, 79.6)
- added C13: 0.1u/25V, Capacitor_SMD:C_0603_1608Metric, F.Cu at (52.0, 81.8)
- added C14: 0.1u/25V, Capacitor_SMD:C_0603_1608Metric, F.Cu at (79.5, 106.9)
- added C15: 0.1u/25V, Capacitor_SMD:C_0603_1608Metric, F.Cu at (55.0, 107.6)
- added C16: 10u/25V, Capacitor_SMD:C_0603_1608Metric, F.Cu at (81.0, 106.9)
- added C17: 10u/25V, Capacitor_SMD:C_0603_1608Metric, F.Cu at (56.5, 107.6)
- added C18: 10u/25V, Capacitor_SMD:C_0603_1608Metric, F.Cu at (82.5, 106.9)
- added C19: 10u/25V, Capacitor_SMD:C_0603_1608Metric, F.Cu at (58.0, 107.6)
- added C2: 0.01u/25V, Capacitor_SMD:C_0603_1608Metric, F.Cu at (104.0, 67.2)
- added C20: 0.1u/25V, Capacitor_SMD:C_0603_1608Metric, F.Cu at (89.4, 102.6)
- added C21: 0.1u/25V, Capacitor_SMD:C_0603_1608Metric, F.Cu at (64.7, 102.6)
- added C22: 22u/16V, Capacitor_SMD:C_1206_3216Metric, F.Cu at (93.1, 100.7)
- added C23: 22u/16V, Capacitor_SMD:C_1206_3216Metric, F.Cu at (68.6, 100.9)
- added C24: 22u/16V, Capacitor_SMD:C_1206_3216Metric, F.Cu at (80.0, 95.6)
- added C25: 22u/16V, Capacitor_SMD:C_1206_3216Metric, F.Cu at (56.3, 95.8)
- added C26: 0.1u/25V, Capacitor_SMD:C_0603_1608Metric, F.Cu at (94.8, 86.3)
- added C27: 0.1u/25V, Capacitor_SMD:C_0603_1608Metric, F.Cu at (67.0, 75.8)
- added C28: 0.1u/25V, Capacitor_SMD:C_0603_1608Metric, F.Cu at (78.8, 80.9)
- added C29: 0.1u/25V, Capacitor_SMD:C_0603_1608Metric, F.Cu at (57.5, 70.1)
- added C3: 0.01u/25V, Capacitor_SMD:C_0603_1608Metric, F.Cu at (42.3, 121.2)
- added C30: 22u/16V Elec, Capacitor_SMD:C_Elec_5x5.8, F.Cu at (78.8, 87.0)
- added C31: 22u/16V Elec, Capacitor_SMD:C_Elec_5x5.8, F.Cu at (63.2, 64.3)
- added C32: 0.1u/25V, Capacitor_SMD:C_0603_1608Metric, F.Cu at (155.7, 100.9)
- added C33: 0.1u/25V, Capacitor_SMD:C_0603_1608Metric, F.Cu at (155.0, 129.4)
- added C34: 0.1u/25V, Capacitor_SMD:C_0603_1608Metric, F.Cu at (181.8, 101.2)
- added C35: 0.1u/25V, Capacitor_SMD:C_0603_1608Metric, F.Cu at (130.4, 95.5)
- added C36: 1uF/16V, Capacitor_SMD:C_0805_2012Metric, F.Cu at (127.7, 92.3)
- added C37: 0.1u/25V, Capacitor_SMD:C_0603_1608Metric, F.Cu at (112.8, 64.5)
- added C38: 10u/25V, Capacitor_SMD:C_0805_2012Metric, F.Cu at (112.8, 66.3)
- added C39: 0.1u/25V, Capacitor_SMD:C_0603_1608Metric, F.Cu at (106.8, 98.3)
- added C4: 0.1u/25V, Capacitor_SMD:C_0603_1608Metric, F.Cu at (106.1, 62.0)
- added C40: 1u/25V, Capacitor_SMD:C_0805_2012Metric, F.Cu at (121.5, 66.0)
- added C41: 0.1u/25V, Capacitor_SMD:C_0603_1608Metric, F.Cu at (111.5, 80.8)
- added C42: 0.1u/25V, Capacitor_SMD:C_0603_1608Metric, F.Cu at (123.9, 83.0)
- added C43: 0.1u/25V, Capacitor_SMD:C_0603_1608Metric, F.Cu at (122.4, 69.2)
- added C44: 0.1u/25V, Capacitor_SMD:C_0603_1608Metric, F.Cu at (110.1, 77.1)
- added C45: 22u/16V Elec, Capacitor_SMD:C_Elec_5x5.8, F.Cu at (105.0, 77.5)
- added C46: DNP, Capacitor_SMD:C_0603_1608Metric, F.Cu at (94.5, 122.3)
- added C47: 0.1u/25V, Capacitor_SMD:C_0603_1608Metric, F.Cu at (98.7, 122.0)
- added C48: 0.1u/25V, Capacitor_SMD:C_0603_1608Metric, F.Cu at (128.3, 105.9)
- added C49: 0.1u/25V, Capacitor_SMD:C_0603_1608Metric, F.Cu at (134.0, 119.0)
- added C5: 0.1u/25V, Capacitor_SMD:C_0603_1608Metric, F.Cu at (59.4, 138.3)
- added C50: 0.1u/25V, Capacitor_SMD:C_0603_1608Metric, F.Cu at (141.7, 129.4)
- added C51: 0.1u/25V, Capacitor_SMD:C_0603_1608Metric, F.Cu at (113.5, 129.8)
- added C52: 0.1u/25V, Capacitor_SMD:C_0603_1608Metric, F.Cu at (133.8, 140.3)
- added C53: 0.1u/25V, Capacitor_SMD:C_0603_1608Metric, F.Cu at (108.4, 114.0)
- added C54: 2.2uF, Capacitor_SMD:C_0603_1608Metric, F.Cu at (139.7, -24.2)
- added C55: 2.2uF, Capacitor_SMD:C_0603_1608Metric, F.Cu at (151.4, -14.9)
- added C56: 0.1u/25V, Capacitor_SMD:C_0603_1608Metric, F.Cu at (139.7, -29.2)
- added C57: 0.1u/25V, Capacitor_SMD:C_0603_1608Metric, F.Cu at (177.8, -6.47)
- added C58: 10uF/10V, Capacitor_SMD:C_0603_1608Metric, F.Cu at (177.8, -31.5)
- added C59: 2.2nF, Capacitor_SMD:C_0603_1608Metric, F.Cu at (151.6, -17.7)
- added C6: 0.1u/25V, Capacitor_SMD:C_0603_1608Metric, F.Cu at (49.4, 66.6)
- added C60: 2.2nF, Capacitor_SMD:C_0603_1608Metric, F.Cu at (142.7, -20.2)
- added C61: 0.1u/25V, Capacitor_SMD:C_0603_1608Metric, F.Cu at (165.1, -35.3)
- added C62: 10uF/10V, Capacitor_SMD:C_0603_1608Metric, F.Cu at (162.1, -38.3)
- added C63: 0.1u/25V, Capacitor_SMD:C_0603_1608Metric, F.Cu at (177.8, -11.5)
- added C64: 4.7uF, Capacitor_SMD:C_0603_1608Metric, F.Cu at (142.7, -15.2)
- added C65: 10uF/10V, Capacitor_SMD:C_0603_1608Metric, F.Cu at (159.4, -23.0)
- added C66: 1u/25V, Capacitor_SMD:C_0805_2012Metric, F.Cu at (150.3, 66.3)
- added C67: 0.47F/5.5V, kicad_gx_library:CP_Supercap_EDC474Z5R5V_0.2x5mm, F.Cu at (135.4, 52.6)
- added C68: 10nF/16V, Capacitor_SMD:C_0603_1608Metric, F.Cu at (147.2, 54.9)
- added C69: 1u/25V, Capacitor_SMD:C_0805_2012Metric, F.Cu at (223.0, 122.7)
- added C7: 0.1u/25V, Capacitor_SMD:C_0603_1608Metric, F.Cu at (49.4, 61.6)
- added C70: 220uF, Capacitor_SMD:CP_Elec_6.3x7.7, F.Cu at (229.0, 136.3)
- added C71: 2.7pF, Capacitor_SMD:C_0603_1608Metric_Pad1.08x0.95mm_HandSolder, F.Cu at (200.9, 61.8)
- added C72: 13pF, Capacitor_SMD:C_0201_0603Metric_Pad0.64x0.40mm_HandSolder, F.Cu at (231.9, 60.8)
- added C73: 12pF, Capacitor_SMD:C_0603_1608Metric_Pad1.08x0.95mm_HandSolder, F.Cu at (199.9, 56.8)
- added C74: 10pF, Capacitor_SMD:C_0603_1608Metric_Pad1.08x0.95mm_HandSolder, F.Cu at (197.9, 62.8)
- added C75: 18pF, Capacitor_SMD:C_0603_1608Metric_Pad1.08x0.95mm_HandSolder, F.Cu at (213.6, 65.9)
- added C76: 16pF, Capacitor_SMD:C_0603_1608Metric_Pad1.08x0.95mm_HandSolder, F.Cu at (210.6, 66.9)
- added C77: 5.1pF, Capacitor_SMD:C_0603_1608Metric_Pad1.08x0.95mm_HandSolder, F.Cu at (229.9, 70.8)
- added C78: 2.2nF, Capacitor_SMD:C_0603_1608Metric_Pad1.08x0.95mm_HandSolder, F.Cu at (196.9, 55.8)
- added C79: 1u/25V, Capacitor_SMD:C_0805_2012Metric, F.Cu at (95.0, 143.6)
- added C8: 0.47u/25V, Capacitor_SMD:C_0805_2012Metric, F.Cu at (47.1, 59.6)
- added C80: 47uF, kicad_gx_library:CP-SMD_1206_L3.2-W1.6-FD, F.Cu at (89.8, 141.6)
- added C81: 0.1u/25V, Capacitor_SMD:C_0603_1608Metric, F.Cu at (85.2, 135.3)
- added C82: 1u/25V, Capacitor_SMD:C_0805_2012Metric, F.Cu at (75.3, 141.6)
- added C83: 0.1u/25V, Capacitor_SMD:C_0603_1608Metric, F.Cu at (104.6, 133.9)
- added C9: 0.47u/10V, Capacitor_SMD:C_0603_1608Metric, F.Cu at (42.4, 67.4)
- added Card1: 472192001, kicad_gx_library:TF-SMD_472192001, F.Cu at (171.4, 105.5)
- added D1: BAS116, kicad_gx_library:SOT-23_L2.9-W1.3-P1.90-LS2.4-BR, F.Cu at (45.0, 137.9)
- added D10: BAS116, kicad_gx_library:SOT-23_L2.9-W1.3-P1.90-LS2.4-BR, F.Cu at (135.7, 65.7)
- added D11: BAS116, kicad_gx_library:SOT-23_L2.9-W1.3-P1.90-LS2.4-BR, F.Cu at (177.2, 111.8)
- added D12: BAS116, kicad_gx_library:SOT-23_L2.9-W1.3-P1.90-LS2.4-BR, F.Cu at (129.7, 61.5)
- added D13: BAS116, kicad_gx_library:SOT-23_L2.9-W1.3-P1.90-LS2.4-BR, F.Cu at (105.7, 137.9)
- added D2: SMAJ18A, Diode_SMD:D_SMA, F.Cu at (54.2, 84.6)
- added D3: WS2812B, LED_SMD:LED_WS2812B_PLCC4_5.0x5.0mm_P3.2mm, F.Cu at (157.4, 105.0)
- added D4: BAS116, kicad_gx_library:SOT-23_L2.9-W1.3-P1.90-LS2.4-BR, F.Cu at (103.8, 127.0)
- added D5: BAS116, kicad_gx_library:SOT-23_L2.9-W1.3-P1.90-LS2.4-BR, F.Cu at (103.8, 123.5)
- added D6: Y, LED_SMD:LED_0805_2012Metric, F.Cu at (108.5, 120.2)
- added D7: BL, LED_SMD:LED_0805_2012Metric, F.Cu at (110.7, 120.1)
- added D8: R, LED_SMD:LED_0805_2012Metric, F.Cu at (112.8, 120.1)
- added D9: G, LED_SMD:LED_0805_2012Metric, F.Cu at (115.1, 120.2)
- added F1: CLM1612P1412, kicad_gx_library:Fuse_PTCC_CLM1612, F.Cu at (48.0, 50.2)
- added F2: Fuse 2A, kicad_gx_library:Fuse_MCCQ-122, F.Cu at (42.0, 129.3)
- added F3: 16V/500mA, Fuse:Fuse_0805_2012Metric, F.Cu at (123.9, 57.4)
- added J1: Conn_01x03, Connector_JST:JST_PH_B3B-PH-SM4-TB_1x03-1MP_P2.00mm_Vertical, F.Cu at (37.8, 138.0)
- added J2: 1377G12-BK, kicad_gx_library:Connector_Anderson_PP25_RA_1377g12-bk, F.Cu at (47.9, 99.4)
- added J3: 236-102, kicad_gx_library:TerminalBlock_WAGO_236-102_1x02_P5.00mm_45Degree, F.Cu at (43.1, 79.8)
- added J4: HC-TYPE-C-16P-01A, Connector_USB:USB_C_Receptacle_HCTL_HC-TYPE-C-16P-01A, F.Cu at (119.5, 49.7)
- added J5: Conn_01x03, Connector_JST:JST_PH_B3B-PH-SM4-TB_1x03-1MP_P2.00mm_Vertical, F.Cu at (164.6, -12.7)
- added J6: Conn_01x03, Connector_JST:JST_PH_B3B-PH-SM4-TB_1x03-1MP_P2.00mm_Vertical, F.Cu at (100.0, 111.8)
- added J7: RF_SMA, Connector_Coaxial:SMA_Amphenol_132289_EdgeMount, F.Cu at (147.2, 48.2)
- added J8: RF_SMA, Connector_Coaxial:SMA_Amphenol_132289_EdgeMount, F.Cu at (186.7, 48.1)
- added J9: AudioJack, kicad_gx_library:Jack_SJ-43617-SMT-TR, F.Cu at (221.9, 103.3)
- added JP1: BATT IN ISO, TestPoint:TestPoint_2Pads_Pitch2.54mm_Drill0.8mm, F.Cu at (40.4, 109.6)
- added JP12: Jumper_2_Open, TestPoint:TestPoint_2Pads_Pitch2.54mm_Drill0.8mm, F.Cu at (69.8, 135.0)
- added JP14: Jumper_2_Open, TestPoint:TestPoint_2Pads_Pitch2.54mm_Drill0.8mm, F.Cu at (69.8, 132.5)
- added JP16: Jumper_2_Open, TestPoint:TestPoint_2Pads_Pitch2.54mm_Drill0.8mm, F.Cu at (98.7, 94.9)
- added JP18: Jumper_2_Open, TestPoint:TestPoint_2Pads_Pitch2.54mm_Drill0.8mm, F.Cu at (98.7, 100.4)
- added JP20: 5V TEST LOAD, TestPoint:TestPoint_2Pads_Pitch2.54mm_Drill0.8mm, F.Cu at (98.7, 74.8)
- added JP21: 3.3V TEST LOAD, TestPoint:TestPoint_2Pads_Pitch2.54mm_Drill0.8mm, F.Cu at (98.8, 64.0)
- added JP22: Jumper_2_Open, TestPoint:TestPoint_2Pads_Pitch2.54mm_Drill0.8mm, F.Cu at (98.7, 80.2)
- added JP24: Jumper_2_Open, TestPoint:TestPoint_2Pads_Pitch2.54mm_Drill0.8mm, F.Cu at (98.8, 69.6)
- added JP26: GND IO0_7, Jumper:SolderJumper-2_P1.3mm_Open_TrianglePad1.0x1.5mm, F.Cu at (92.0, 110.6)
- added JP27: Write Protect, Jumper:SolderJumper-2_P1.3mm_Open_TrianglePad1.0x1.5mm, B.Cu at (130.2, 103.2)
- added JP28: Bypass PWR SW, TestPoint:TestPoint_2Pads_Pitch2.54mm_Drill0.8mm, F.Cu at (154.6, 64.3)
- added JP29: TX Watchdog Bypass, Jumper:SolderJumper-2_P1.3mm_Open_TrianglePad1.0x1.5mm, F.Cu at (82.5, 135.2)
- added JP3: 12V IN ISO, TestPoint:TestPoint_2Pads_Pitch2.54mm_Drill0.8mm, F.Cu at (43.0, 109.6)
- added JP5: 5V SEL BYPASS, TestPoint:TestPoint_2Pads_Pitch2.54mm_Drill0.8mm, F.Cu at (98.8, 86.8)
- added JP6: PWR ISO, TestPoint:TestPoint_2Pads_Pitch2.54mm_Drill0.8mm, F.Cu at (66.7, 132.5)
- added JP8: 3.3V SEL BYPASS, TestPoint:TestPoint_2Pads_Pitch2.54mm_Drill0.8mm, F.Cu at (109.5, 72.4)
- added JP9: MAIN SW BYPASS, TestPoint:TestPoint_2Pads_Pitch2.54mm_Drill0.8mm, F.Cu at (57.5, 127.4)
- added L1: 3.3uH, kicad_gx_library:L_Chilisin_MHCI06030, F.Cu at (85.3, 96.9)
- added L2: 3.3uH, kicad_gx_library:L_Chilisin_MHCI06030, F.Cu at (61.0, 96.9)
- added L3: 27nH, Inductor_SMD:L_0402_1005Metric, F.Cu at (145.4, 54.1)
- added L4: 43nH, Inductor_SMD:L_0805_2012Metric_Pad1.05x1.20mm_HandSolder, F.Cu at (225.9, 54.8)
- added L5: 30nH, Inductor_SMD:L_0805_2012Metric_Pad1.05x1.20mm_HandSolder, F.Cu at (222.9, 54.8)
- added L6: 27nH, Inductor_SMD:L_0805_2012Metric_Pad1.05x1.20mm_HandSolder, F.Cu at (219.9, 54.8)
- added L7: ~, Inductor_SMD:L_0603_1608Metric, F.Cu at (226.9, 59.8)
- added L8: ~, Inductor_SMD:L_0603_1608Metric, F.Cu at (229.9, 60.8)
- added L9: ~, Inductor_SMD:L_0603_1608Metric, F.Cu at (210.9, 54.8)
- added Q1: AO3407A, Package_TO_SOT_SMD:SOT-23, F.Cu at (52.9, 130.2)
- added Q10: BSS138, Package_TO_SOT_SMD:SOT-23, F.Cu at (145.2, 72.4)
- added Q11: AO3407A, Package_TO_SOT_SMD:SOT-23, F.Cu at (150.5, 71.6)
- added Q12: BSS138, Package_TO_SOT_SMD:SOT-23, F.Cu at (234.1, 126.0)
- added Q13: BSS138, Package_TO_SOT_SMD:SOT-23, F.Cu at (228.9, 125.5)
- added Q14: BSS138, Package_TO_SOT_SMD:SOT-23, F.Cu at (105.6, 142.0)
- added Q2: AO3400A, Package_TO_SOT_SMD:SOT-23, F.Cu at (40.5, 52.5)
- added Q3: 8205A, digikey-kicad-library:SOT23-6L, F.Cu at (44.5, 55.2)
- added Q4: BSS138, Package_TO_SOT_SMD:SOT-23, F.Cu at (65.0, 128.7)
- added Q5: BSS138, Package_TO_SOT_SMD:SOT-23, F.Cu at (65.0, 137.8)
- added Q6: MMBT2222A, Package_TO_SOT_SMD:SOT-23, F.Cu at (116.7, 87.8)
- added Q7: MMBT2222A, Package_TO_SOT_SMD:SOT-23, F.Cu at (110.5, 88.0)
- added Q8: AO3407A, Package_TO_SOT_SMD:SOT-23, F.Cu at (82.3, 127.7)
- added Q9: BSS138, Package_TO_SOT_SMD:SOT-23, F.Cu at (69.9, 128.7)
- added R1: 5k, Resistor_SMD:R_0201_0603Metric, F.Cu at (37.9, 115.8)
- added R10: 1M, Resistor_SMD:R_0603_1608Metric, F.Cu at (44.3, 134.0)
- added R11: 1M, Resistor_SMD:R_0603_1608Metric, F.Cu at (56.9, 132.9)
- added R12: 10, Resistor_SMD:R_0805_2012Metric, F.Cu at (49.2, 56.9)
- added R13: 150, Resistor_SMD:R_1206_3216Metric, F.Cu at (51.1, 63.8)
- added R14: 150, Resistor_SMD:R_1206_3216Metric, F.Cu at (55.6, 59.3)
- added R15: 0.0025, kicad_gx_library:RES-SMD_L6.4-W3.2-R2512_Sense4Pin, F.Cu at (46.1, 71.8)
- added R16: 1k, Resistor_SMD:R_0805_2012Metric, F.Cu at (40.8, 59.5)
- added R17: 820, Resistor_SMD:R_0805_2012Metric, F.Cu at (43.0, 59.5)
- added R18: 10k, Resistor_SMD:R_0603_1608Metric, F.Cu at (86.4, 107.9)
- added R19: 10k, Resistor_SMD:R_0603_1608Metric, F.Cu at (62.1, 108.1)
- added R2: 23.7k, Resistor_SMD:R_0603_1608Metric, F.Cu at (45.6, 112.5)
- added R20: 10k, Resistor_SMD:R_0603_1608Metric, F.Cu at (89.4, 106.3)
- added R21: 10k, Resistor_SMD:R_0603_1608Metric, F.Cu at (64.8, 106.7)
- added R22: 76.8k, Resistor_SMD:R_0603_1608Metric, F.Cu at (91.0, 104.7)
- added R23: 52.3k, Resistor_SMD:R_0603_1608Metric, F.Cu at (66.4, 105.0)
- added R24: 24.9 2W, Resistor_THT:R_Axial_Power_L20.0mm_W6.4mm_P5.08mm_Vertical, F.Cu at (108.7, 53.5)
- added R25: 16.5 2W, Resistor_THT:R_Axial_Power_L20.0mm_W6.4mm_P5.08mm_Vertical, F.Cu at (101.5, 53.5)
- added R26: 10k, Resistor_SMD:R_0603_1608Metric, F.Cu at (69.7, 137.9)
- added R27: 10k, Resistor_SMD:R_0603_1608Metric, F.Cu at (181.4, 105.5)
- added R28: 10k, Resistor_SMD:R_0603_1608Metric, F.Cu at (151.7, 134.4)
- added R29: 10k, Resistor_SMD:R_0603_1608Metric, F.Cu at (155.2, 134.5)
- added R3: 23.7k, Resistor_SMD:R_0603_1608Metric, F.Cu at (37.9, 112.9)
- added R30: 5.1k, Resistor_SMD:R_0603_1608Metric, F.Cu at (120.7, 57.2)
- added R31: 5.1k, Resistor_SMD:R_0603_1608Metric, F.Cu at (117.7, 57.2)
- added R32: 10k, Resistor_SMD:R_0603_1608Metric, F.Cu at (116.1, 90.4)
- added R33: 10k, Resistor_SMD:R_0603_1608Metric, F.Cu at (113.8, 88.0)
- added R34: 10k, Resistor_SMD:R_0603_1608Metric, F.Cu at (119.6, 87.8)
- added R35: 10k, Resistor_SMD:R_0603_1608Metric, F.Cu at (91.1, 127.7)
- added R36: 100k, Resistor_SMD:R_0603_1608Metric, F.Cu at (74.5, 128.2)
- added R37: 750, Resistor_SMD:R_0603_1608Metric, F.Cu at (108.5, 123.7)
- added R38: 330, Resistor_SMD:R_0603_1608Metric, F.Cu at (110.7, 123.7)
- added R39: 590, Resistor_SMD:R_0603_1608Metric, F.Cu at (112.8, 123.7)
- added R4: 5k, Resistor_SMD:R_0201_0603Metric, F.Cu at (41.7, 113.9)
- added R40: 330, Resistor_SMD:R_0603_1608Metric, F.Cu at (115.1, 123.6)
- added R41: 10k, Resistor_SMD:R_0603_1608Metric, F.Cu at (115.9, 114.0)
- added R42: 10k, Resistor_SMD:R_0603_1608Metric, F.Cu at (165.1, -24.2)
- added R43: 470, Resistor_SMD:R_0603_1608Metric, F.Cu at (152.4, -9.88)
- added R44: 470, Resistor_SMD:R_0603_1608Metric, F.Cu at (151.6, -22.7)
- added R45: 100k, Resistor_SMD:R_0603_1608Metric, F.Cu at (142.6, -35.7)
- added R46: 150, Resistor_SMD:R_0603_1608Metric, F.Cu at (145.7, -17.2)
- added R47: 10k, Resistor_SMD:R_0603_1608Metric, F.Cu at (102.1, 58.1)
- added R48: 10k, Resistor_SMD:R_0603_1608Metric, F.Cu at (121.0, 120.3)
- added R49: 10k, Resistor_SMD:R_0603_1608Metric, F.Cu at (141.7, 72.2)
- added R5: 30.1k, Resistor_SMD:R_0603_1608Metric, F.Cu at (104.1, 92.5)
- added R50: 10k, Resistor_SMD:R_0603_1608Metric, F.Cu at (137.1, 70.4)
- added R51: 1M, Resistor_SMD:R_0603_1608Metric, F.Cu at (149.6, 75.6)
- added R52: 10, Resistor_SMD:R_1206_3216Metric, F.Cu at (142.0, 54.1)
- added R53: 10, Resistor_SMD:R_0603_1608Metric, F.Cu at (131.2, 56.7)
- added R54: 10k, Resistor_SMD:R_0603_1608Metric, F.Cu at (225.7, 127.8)
- added R55: 10k, Resistor_SMD:R_0603_1608Metric, F.Cu at (67.1, 124.8)
- added R56: 0, Resistor_SMD:R_0603_1608Metric, F.Cu at (226.9, 66.8)
- added R57: 0, Resistor_SMD:R_0603_1608Metric, F.Cu at (229.9, 65.8)
- added R58: 0, Resistor_SMD:R_0603_1608Metric, F.Cu at (207.9, 54.8)
- added R59: 10k, Resistor_SMD:R_0603_1608Metric, F.Cu at (238.4, 118.5)
- added R6: 10k, Resistor_SMD:R_0603_1608Metric, F.Cu at (102.5, 92.5)
- added R60: 470k, Resistor_SMD:R_0603_1608Metric, F.Cu at (86.8, 142.2)
- added R61: 10k, Resistor_SMD:R_0603_1608Metric, F.Cu at (80.8, 143.2)
- added R62: 10k, Resistor_SMD:R_0603_1608Metric, F.Cu at (74.8, 137.9)
- added R63: 10k, Resistor_SMD:R_0603_1608Metric, F.Cu at (101.2, 143.8)
- added R64: 10k, Resistor_SMD:R_0603_1608Metric, F.Cu at (238.2, 126.9)
- added R65: 10k, Resistor_SMD:R_0603_1608Metric, F.Cu at (109.2, 142.1)
- added R66: 10k, Resistor_SMD:R_0603_1608Metric, F.Cu at (229.3, 129.8)
- added R67: 10k, Resistor_SMD:R_0603_1608Metric, F.Cu at (106.6, 133.8)
- added R68: 10k, Resistor_SMD:R_0603_1608Metric, F.Cu at (128.7, 131.9)
- added R69: 10k, Resistor_SMD:R_0603_1608Metric, F.Cu at (126.3, 128.3)
- added R7: 80.6k, Resistor_SMD:R_0603_1608Metric, F.Cu at (105.7, 67.2)
- added R70: 10k, Resistor_SMD:R_0603_1608Metric, F.Cu at (120.9, 140.0)
- added R71: 10k, Resistor_SMD:R_0603_1608Metric, F.Cu at (93.2, 114.5)
- added R8: 30.1k, Resistor_SMD:R_0603_1608Metric, F.Cu at (40.7, 121.2)
- added R9: 10k, Resistor_SMD:R_0603_1608Metric, F.Cu at (107.2, 67.2)
- added RV1: 1k, Potentiometer_SMD:Potentiometer_Bourns_3314G_Vertical, F.Cu at (148.6, -31.7)
- added SW1: POWER, Button_Switch_SMD:SW_SPST_PTS645Sx43SMTR92, F.Cu at (53.1, 138.6)
- added SW2: RST, Button_Switch_SMD:SW_SPST_PTS645Sx43SMTR92, F.Cu at (124.4, 96.9)
- added SW3: BOOT, Button_Switch_SMD:SW_SPST_PTS645Sx43SMTR92, F.Cu at (113.0, 96.9)
- added SW4: GENERAL, Button_Switch_SMD:SW_SPST_PTS645Sx43SMTR92, F.Cu at (127.5, 120.0)
- added SW5: GENERAL, Button_Switch_SMD:SW_SPST_PTS645Sx43SMTR92, F.Cu at (135.0, 130.0)
- added SW6: GENERAL, Button_Switch_SMD:SW_SPST_PTS645Sx43SMTR92, F.Cu at (120.0, 130.0)
- added SW7: GENERAL, Button_Switch_SMD:SW_SPST_PTS645Sx43SMTR92, F.Cu at (127.5, 140.0)
- added SW8: SW_DIP_x04, Button_Switch_SMD:SW_DIP_SPSTx04_Slide_KingTek_DSHP04TS_W7.62mm_P1.27mm, F.Cu at (122.2, 108.9)
- added SW9: NSI-10S, kicad_gx_library:SW-SMD_NSI-10S, F.Cu at (128.3, 51.1)
- added TH1: NCP15XH103F03RC, Resistor_SMD:R_0402_1005Metric, F.Cu at (40.7, 63.8)
- added U1: TPS2121RUXR, kicad_gx_library:VQFN-HR-12_L2.5-W2.0-P0.50-BL, F.Cu at (103.1, 88.2)
- added U10: ESP32-S3-WROOM-1-N8R8, RF_Module:ESP32-S3-WROOM-1, F.Cu at (170.4, 132.0)
- added U11: CH334R, Package_SO:QSOP-16_3.9x4.9mm_P0.635mm, F.Cu at (117.7, 64.1)
- added U12: CH340C, Package_SO:SOIC-16_3.9x9.9mm_P1.27mm, F.Cu at (117.7, 80.8)
- added U13: LM1117IMPX-3.3, Package_TO_SOT_SMD:SOT-223-3_TabPin2, F.Cu at (115.8, 72.4)
- added U14: CAT24C32YI-GT3, kicad_gx_library:TSSOP-8_L4.4-W3.0-P0.65-LS6.4-BL, F.Cu at (131.1, 109.3)
- added U15: PCF8563T, Package_SO:SOIC-8_3.9x4.9mm_P1.27mm, F.Cu at (97.0, 126.0)
- added U16: PCA9555PW, Package_SO:TSSOP-24_4.4x7.8mm_P0.65mm, F.Cu at (112.3, 108.6)
- added U17: PCM5102A, Package_SO:TSSOP-20_4.4x6.5mm_P0.65mm, F.Cu at (154.6, -10.7)
- added U19: MAX-M10S, RF_GPS:ublox_MAX, F.Cu at (143.8, 63.2)
- added U2: TPS2121RUXR, kicad_gx_library:VQFN-HR-12_L2.5-W2.0-P0.50-BL, F.Cu at (104.8, 71.2)
- added U20: SA818S-V, kicad_gx_library:WIRELM-SMD_G-NICERF_SA818S-X, F.Cu at (201.8, 115.0)
- added U21: 74HC123, Package_SO:SOIC-16_3.9x9.9mm_P1.27mm, F.Cu at (98.7, 137.2)
- added U23: 74LVC1G38, Package_TO_SOT_SMD:SOT-23-5, F.Cu at (78.8, 138.9)
- added U24: 74LVC1G38, Package_TO_SOT_SMD:SOT-23-5, F.Cu at (83.9, 138.8)
- added U25: 74LVC1G38, Package_TO_SOT_SMD:SOT-23-5, F.Cu at (106.1, 59.2)
- added U3: TPS2121RUXR, kicad_gx_library:VQFN-HR-12_L2.5-W2.0-P0.50-BL, F.Cu at (41.7, 117.3)
- added U5: MAX17320, Package_DFN_QFN:TQFN-24-1EP_4x4mm_P0.5mm_EP2.1x2.1mm, F.Cu at (45.0, 63.9)
- added U6: TPS563201, Package_TO_SOT_SMD:SOT-23-6, F.Cu at (86.1, 104.5)
- added U7: TPS563201, Package_TO_SOT_SMD:SOT-23-6, F.Cu at (61.8, 104.6)
- added U8: LM1085-5.0, Package_TO_SOT_SMD:TO-263-3_TabPin2, F.Cu at (87.8, 81.3)
- added U9: LM1117IMPX-3.3, Package_TO_SOT_SMD:SOT-223-3_TabPin2, F.Cu at (62.1, 73.0)
- added X1: 12MHz 10pF, kicad_gx_library:CRYSTAL-SMD_4P-L2.5-W2.0-BL, F.Cu at (112.5, 62.0)
- added Y2: 32.768kHz 9pF, Crystal:Crystal_SMD_3215-2Pin_3.2x1.5mm, F.Cu at (91.5, 123.8)
Routing:
- net GND: track 0.00 -> 211.9 mm, vias 0 -> 114
- net /Peripherals/PERIPH_SCL: track 0.00 -> 136.3 mm, vias 0 -> 6
- net /Peripherals/PERIPH_SDA: track 0.00 -> 135.7 mm, vias 0 -> 4
- net /Power/Battery 18650 Input/BATT_Plus_to_Minus: track 0.00 -> 122.9 mm
- net /Power/Battery 18650 Input/PWR_18650: track 0.00 -> 64.3 mm
- net Net-(U16-IO1_2): track 0.00 -> 62.8 mm
- net /Power/Battery_PowerPole_Input/PWR_POWERPOLE: track 0.00 -> 57.3 mm
- net Net-(U16-IO1_0): track 0.00 -> 56.7 mm, vias 0 -> 2
- net /GPS/GPS_IN_PWRON: track 0.00 -> 55.4 mm
- net +3.3V: track 0.00 -> 54.9 mm, vias 0 -> 31
- net /Power/Power Regulation/3V3_BUCK_OUT: track 0.00 -> 54.3 mm, vias 0 -> 1
- net /Power/Power Regulation/3V3_LDO_OUT: track 0.00 -> 54.0 mm
- net /Power/Power Regulation/3V3_LDO_VIN: track 0.00 -> 52.1 mm, vias 0 -> 1
- net /Peripherals/RTC_OUT_INTERRUPT_LATCH: track 0.00 -> 45.6 mm, vias 0 -> 2
- net /Power/Power Regulation/3V3_BUCK_VIN: track 0.00 -> 45.5 mm
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- added copper zone on F.Cu, net +3.3V
- added copper zone on F.Cu, net +5V
- added copper zone on F.Cu, net /Power/BATT_IN1
- added copper zone on F.Cu, net /Power/BATT_IN2
- added copper zone on F.Cu, net /Power/BATT_MUX_OUT
- added copper zone on F.Cu, net /Power/Power Regulation/BATT_3.3V_REG
- added copper zone on F.Cu, net /Power/Power Regulation/BATT_5V_REG
- added copper zone on F.Cu, net /Power/USB_3.3V_IN
- added copper zone on F.Cu, net /Power/USB_5V_SW
Other:
- board outline added: 214.1 x 100 mm

Commit message: blocks
Parts:
- moved J8 371.6 mm to (531.4, -90.7)
- moved C71 371.6 mm to (545.6, -77.0)
- moved C72 371.6 mm to (576.6, -78.0)
- moved C73 371.6 mm to (544.6, -82.0)
- moved C74 371.6 mm to (542.6, -76.0)
- moved C75 371.6 mm to (558.2, -72.9)
- moved C76 371.6 mm to (555.2, -71.9)
- moved C77 371.6 mm to (574.6, -68.0)
- moved C78 371.6 mm to (541.6, -83.0)
- moved L4 371.6 mm to (570.6, -84.0)
- moved L5 371.6 mm to (567.6, -84.0)
- moved L6 371.6 mm to (564.6, -84.0)
- moved L7 371.6 mm to (571.6, -79.0)
- moved L8 371.6 mm to (574.6, -78.0)
- moved L9 371.6 mm to (555.6, -84.0)
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Routing:
- net GND: track 211.9 -> 0.00 mm, vias 114 -> 0
- net /Peripherals/PERIPH_SCL: track 136.3 -> 0.00 mm, vias 6 -> 0
- net /Peripherals/PERIPH_SDA: track 135.7 -> 0.00 mm, vias 4 -> 0
- net /Power/Battery 18650 Input/PWR_18650: track 64.3 -> 10.5 mm
- net /GPS/GPS_IN_PWRON: track 55.4 -> 2.61 mm
- net /Peripherals/RTC_OUT_INTERRUPT_LATCH: track 45.6 -> 0.00 mm, vias 2 -> 0
- net Net-(U1-ST): track 41.6 -> 0.00 mm, vias 2 -> 0
- net /Power/Power Regulation/3V3_LDO_VIN: track 52.1 -> 12.5 mm, vias 1 -> 0
- net +3.3V: track 54.9 -> 16.6 mm, vias 31 -> 0
- net /Power/POWER_PB_SIGNAL: track 35.5 -> 0.00 mm
- net Net-(U16-IO1_2): track 62.8 -> 27.6 mm
- net /Power/Power Regulation/3V3_BUCK_OUT: track 54.3 -> 20.0 mm, vias 1 -> 0
- net /Power/Power Regulation/5V_BUCK_VIN: track 44.8 -> 11.6 mm
- net /Power/BATT_MUX_OUT: track 32.2 -> 0.00 mm
- net /Power/USB_3.3V_IN: track 30.9 -> 0.00 mm, vias 4 -> 0
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- added copper zone on F.Cu, net GNDREF
- removed copper zone on F.Cu, net +3.3V
- removed copper zone on F.Cu, net +5V
- removed copper zone on F.Cu, net /Power/Power Regulation/BATT_3.3V_REG
- removed copper zone on F.Cu, net /Power/Power Regulation/BATT_5V_REG
- removed copper zone on F.Cu, net /Power/USB_3.3V_IN
- removed copper zone on F.Cu, net /Power/USB_5V_SW
Other:
- board outline removed
- board text added: "1 10K UP 2 P07 3 GND"
- board text added: "1 P00 2 P01 3 P02 4 P03"
- board text added: "12V INPUT 14.5V MAX 3A MAX"
- board text added: "2.5mΩ"
- board text added: "2S1P 18650s 7.4V nom / 8.4V max"
- board text added: "ALRT GPIO2 I2C SDA GPIO8 I2C SCL GPIO9 I2C ADDR 0x6C MEM 0x000-0FF 0x16 MEM 0x180-1FF"
- board text added: "BATTERY REGULATION 4.8V INTERMEDIATE 5V LDO 1AMP"
- board text added: "BATTERY REGULATION 6.6V INTERMEDIATE 5V LDO 2AMP"
- board text added: "D9 GREEN P14 D8 RED P15 D7 BLUE P16 D6 YELLOW P17"
- board text added: "GND"
- board text added: "GPS uBLOX MAX-M10S"
- board text added: "LRCK GPIO21 DIN GPIO47 BCK GPIO14 XSMT GPIO3"
- board text added: "MAX17230"
- board text added: "OUTR"
- board text added: "P04 SA818 PD P05 SA818 HI/LO P06 GPS PWR SW"
- board text added: "PCA9555 I2C IO EXPANDER I2C ADDR 0x20"
- board text added: "PCM5102A I2S AUDIO"
- board text added: "SW7 DOWN P10 SW6 LEFT P11 SW5 RIGHT P12 SW4 UP P13"
- board text added: "UART TXD GPIO44 UART RXD GPIO43 EXTINT IN GPIO4 -> BATT SW Q1 GPS 1PPS GPIO5 GPS PWR IO P06"
- board text added: "onSemi CAT24C32YI-GT3 32Kb EEPROM I2C ADDR 0xA0 WRITE I2C ADDR 0xA1 READ"

Commit message: module routing
Parts:
- J7, J8: footprint Connector_Coaxial:SMA_Amphenol_132289_EdgeMount -> Connector_Coaxial:SMA_Amphenol_132134-11_Vertical
- moved C69 516.6 mm to (80.7, 189.2)
- moved C70 516.6 mm to (86.7, 202.8)
- moved C75 516.6 mm to (111.7, 186.7)
- moved C76 516.6 mm to (108.7, 187.7)
- moved J8 516.6 mm to (84.8, 168.9)
- moved Q13 516.6 mm to (86.6, 192.1)
- moved C71 516.6 mm to (99.1, 182.6)
- moved C72 516.6 mm to (130.1, 181.6)
- moved C73 516.6 mm to (98.1, 177.6)
- moved C74 516.6 mm to (96.1, 183.6)
- moved C77 516.6 mm to (128.1, 191.6)
- moved C78 516.6 mm to (95.1, 176.6)
- moved L4 516.6 mm to (124.1, 175.6)
- moved L5 516.6 mm to (121.1, 175.6)
- moved L6 516.6 mm to (118.1, 175.6)
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Routing:
- net /USB-C/USB_5V_Fused: track 0.00 -> 49.0 mm, vias 0 -> 2
- net /USB-C/MCU_EN_RESET: track 0.00 -> 42.3 mm, vias 0 -> 2
- net /SA818S-V/SA818_IN_PTT: track 0.00 -> 29.6 mm
- net /Power/BATT_MUX_OUT: track 0.00 -> 27.5 mm, vias 4 -> 8
- net /Power/POWER_PB_SIGNAL: track 0.00 -> 23.4 mm
- net /Power/USB_3.3V_IN: track 0.00 -> 21.9 mm, vias 0 -> 1
- net /Peripherals/RTC_OUT_INTERRUPT_LATCH: track 0.00 -> 19.9 mm
- net +3.3V: track 16.6 -> 33.0 mm, vias 0 -> 2
- net /USB-C/MCU_IO0_BOOT: track 0.00 -> 16.3 mm
- net Net-(U21A-RCext): track 0.00 -> 16.1 mm
- net /USB-C/USB_5V: track 0.00 -> 13.1 mm
- net /Peripherals/RTC_OUT_MCU_INT_ALRM: track 0.00 -> 13.1 mm
- net /Power/POWER_PRESWITCH: track 0.00 -> 13.0 mm
- net Net-(Q8-S): track 0.00 -> 12.1 mm
- net Net-(Card1-DAT0): track 0.00 -> 11.8 mm
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- added copper zone on F.Cu, net +3.3V
- added copper zone on F.Cu, net +5V
- added copper zone on F.Cu, net /Power/Power Regulation/BATT_3.3V_REG
- added copper zone on F.Cu, net /Power/Power Regulation/BATT_5V_REG
- added copper zone on F.Cu, net /Power/USB_3.3V_IN
- added copper zone on F.Cu, net /Power/USB_5V_SW
Other:
- board outline added: 191.5 x 121.8 mm
- board text added: "ALRM INT GPIO1"
- board text added: "BATTERY MUX & POWER ON SWITCH"
- board text added: "BATTERY REGULATION 4.8V INTERMEDIATE 3.3V LDO 1AMP"
- board text added: "BOOT"
- board text added: "CAT24C32YI-GT3 32Kb EEPROM I2C ADDR 0xA0 WR I2C ADDR 0xA1 RD"
- board text added: "ESP32-S3 MCU"
- board text added: "I2C ADDR 0xA2 RD ADDR 0xA3 WR"
- board text added: "POWER BTN GPIO38 PWR LATCH GPIO48 -> RTC INT PIN 3"
- board text added: "POWER SW"
- board text added: "PTT HB GPIO15 PTT GPIO16"
- board text added: "RST"
- board text added: "RTC"
- board text added: "SD CARD SDIO GPIO10 SDO GPIO11 CMD GPIO12 CLK GPIO13 DAT0"
- board text added: "TX WATCHDOG"
- board text added: "Tpw = (0.45)(47uF)(470k) = 9.45sec"
- board text added: "USB-C"
- board text added: "WS2812B GPIO40"
- board text removed: "12V INPUT 14.5V MAX 3A MAX"
- board text removed: "BATTERY REGULATION 4.8V INTERMEDIATE 5V LDO 1AMP"
- board text removed: "onSemi CAT24C32YI-GT3 32Kb EEPROM I2C ADDR 0xA0 WRITE I2C ADDR 0xA1 READ"
